File: 7.0/projects/BrevIce PCBA/BrevIce PCBA/BrevIce PCBA.kicad_pcb (KiCad board)
At the start: 2 copper layers, 120 x 70 mm, 9 parts, among them J1 Conn_01x04_Socket, J2 Conn_01x05_Socket, K1 Relay_SPDT, K2 Relay_SPDT, Q1 AO3400A, Q2 AO3400A, U1 ATmega3208-X

Commit message: Update BrevIce PCBA.kicad_pcb
Parts:
- added DS1: NHD-0420AZ-FL-YBW-33V3, SamacSys_Parts:NHD0420AZFLYBW33V3, F.Cu at (86.4, 59.8)
- added R1: 4.7K, Resistor_SMD:R_0603_1608Metric_Pad0.98x0.95mm_HandSolder, F.Cu at (77.0, 107.1)
Connections:
- U1 pad 19: unconnected-(U1-UPDI-Pad19) -> Net-(U1-UPDI)
- U1 pad 20: unconnected-(U1-VDD-Pad20) -> Net-(J3-Pin_1)

Commit message: Update
Parts:
- moved DS1 6.39 mm to (90.4, 64.8)
Connections:
- DS1 pad 1: unconnected-(DS1-VSS-Pad1) -> +5V
- DS1 pad 10: unconnected-(DS1-DB3-Pad10) -> Net-(DS1-DB3)
- DS1 pad 11: unconnected-(DS1-DB4-Pad11) -> Net-(DS1-DB4)
- DS1 pad 12: unconnected-(DS1-DB5-Pad12) -> Net-(DS1-DB5)
- DS1 pad 13: unconnected-(DS1-DB6-Pad13) -> Net-(DS1-DB6)
- DS1 pad 14: unconnected-(DS1-DB7-Pad14) -> Net-(DS1-DB7)
- DS1 pad 2: unconnected-(DS1-VDD-Pad2) -> GND
- DS1 pad 7: unconnected-(DS1-DB0-Pad7) -> Net-(DS1-DB0)
- DS1 pad 8: unconnected-(DS1-DB1-Pad8) -> Net-(DS1-DB1)
- DS1 pad 9: unconnected-(DS1-DB2-Pad9) -> Net-(DS1-DB2)
- DS1 pad MH1: unconnected-(DS1-PadMH1) -> GND
- DS1 pad MH2: unconnected-(DS1-PadMH2) -> GND
- DS1 pad MH3: unconnected-(DS1-PadMH3) -> GND
- DS1 pad MH4: unconnected-(DS1-PadMH4) -> GND
- U1 pad 24: Net-(J1-Pin_2) -> Net-(U1-PA2)
- U1 pad 25: Net-(J1-Pin_3) -> Net-(U1-PA3)
Changed lines of the file:
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@@
   (net 28 "unconnected-(U1-PF1{slash}TOSC2-Pad17)")
   (net 29 "unconnected-(U1-PF6{slash}~{RESET}-Pad18)")
-  (net 30 "unconnected-(DS1-VSS-Pad1)")
-  (net 31 "unconnected-(DS1-VDD-Pad2)")
+  (net 30 "Net-(DS1-DB0)")
+  (net 31 "Net-(DS1-DB1)")
   (net 32 "unconnected-(U1-EXTCLK{slash}PA0-Pad22)")
   (net 33 "unconnected-(U1-PA1-Pad23)")
@@
   (net 39 "unconnected-(DS1-R{slash}W-Pad5)")
   (net 40 "unconnected-(DS1-E-Pad6)")
-  (net 41 "unconnected-(DS1-DB0-Pad7)")
-  (net 42 "unconnected-(DS1-DB1-Pad8)")
-  (net 43 "unconnected-(DS1-DB2-Pad9)")
-  (net 44 "unconnected-(DS1-DB3-Pad10)")
-  (net 45 "unconnected-(DS1-DB4-Pad11)")
-  (net 46 "unconnected-(DS1-DB5-Pad12)")
-  (net 47 "unconnected-(DS1-DB6-Pad13)")
-  (net 48 "unconnected-(DS1-DB7-Pad14)")
+  (net 41 "Net-(DS1-DB2)")
+  (net 42 "Net-(DS1-DB3)")
+  (net 43 "Net-(DS1-DB4)")
+  (net 44 "Net-(DS1-DB5)")
+  (net 45 "Net-(DS1-DB6)")
+  (net 46 "Net-(DS1-DB7)")
+  (net 47 "Net-(U1-PA2)")
+  (net 48 "Net-(U1-PA3)")
   (net 49 "unconnected-(DS1-LED+-Pad15)")
   (net 50 "unconnected-(DS1-LED--Pad16)")
-  (net 51 "unconnected-(DS1-PadMH1)")
-  (net 52 "unconnected-(DS1-PadMH2)")
-  (net 53 "unconnected-(DS1-PadMH3)")
-  (net 54 "unconnected-(DS1-PadMH4)")
-  (net 55 "Net-(U1-UPDI)")
-  (net 56 "Net-(J3-Pin_3)")
-  (net 57 "Net-(J3-Pin_1)")
+  (net 51 "Net-(U1-UPDI)")
+  (net 52 "Net-(J3-Pin_3)")
+  (net 53 "Net-(J3-Pin_1)")
   (footprint "Package_SO:SSOP-28_5.3x10.2mm_P0.65mm" (layer "F.Cu")
     (at 134.62 83.82 90)
@@
       (net 29 "unconnected-(U1-PF6{slash}~{RESET}-Pad18)") (pinfunction "PF6/~{RESET}") (pintype "bidirectional"))
     (pad "19" smd rect (at 3.6 1.625 90) (size 1.75 0.45) (layers "F.Cu" "F.Paste" "F.Mask")
-      (net 55 "Net-(U1-UPDI)") (pinfunction "UPDI") (pintype "bidirectional"))
+      (net 51 "Net-(U1-UPDI)") (pinfunction "UPDI") (pintype "bidirectional"))
     (pad "20" smd rect (at 3.6 0.975 90) (size 1.75 0.45) (layers "F.Cu" "F.Paste" "F.Mask")
-      (net 57 "Net-(J3-Pin_1)") (pinfunction "VDD") (pintype "power_in"))
+      (net 53 "Net-(J3-Pin_1)") (pinfunction "VDD") (pintype "power_in"))
     (pad "21" smd rect (at 3.6 0.325 90) (size 1.75 0.45) (layers "F.Cu" "F.Paste" "F.Mask")
       (net 26 "GND") (pinfunction "GND") (pintype "passive"))
@@
       (net 33 "unconnected-(U1-PA1-Pad23)") (pinfunction "PA1") (pintype "bidirectional"))
     (pad "24" smd rect (at 3.6 -1.625 90) (size 1.75 0.45) (layers "F.Cu" "F.Paste" "F.Mask")
-      (net 6 "Net-(J1-Pin_2)") (pinfunction "PA2") (pintype "bidirectional"))
+      (net 47 "Net-(U1-PA2)") (pinfunction "PA2") (pintype "bidirectional"))
     (pad "25" smd rect (at 3.6 -2.275 90) (size 1.75 0.45) (layers "F.Cu" "F.Paste" "F.Mask")
-      (net 7 "Net-(J1-Pin_3)") (pinfunction "PA3") (pintype "bidirectional"))
+      (net 48 "Net-(U1-PA3)") (pinfunction "PA3") (pintype "bidirectional"))
     (pad "26" smd rect (at 3.6 -2.925 90) (size 1.75 0.45) (layers "F.Cu" "F.Paste" "F.Mask")
       (net 34 "unconnected-(U1-PA4-Pad26)") (pinfunction "PA4") (pintype "bidirectional"))
@@
       (stroke (width 0.1) (type solid)) (layer "F.Fab"))
     (pad "1" smd roundrect (at -0.9125 0) (size 0.975 0.95) (layers "F.Cu" "F.Paste" "F.Mask") (roundrect_rratio 0.25)
-      (net 55 "Net-(U1-UPDI)") (pintype "passive"))
+      (net 51 "Net-(U1-UPDI)") (pintype "passive"))
     (pad "2" smd roundrect (at 0.9125 0) (size 0.975 0.95) (layers "F.Cu" "F.Paste" "F.Mask") (roundrect_rratio 0.25)
-      (net 56 "Net-(J3-Pin_3)") (pintype "passive"))
+      (net 52 "Net-(J3-Pin_3)") (pintype "passive"))
     (model "${KICAD6_3DMODEL_DIR}/Resistor_SMD.3dshapes/R_0603_1608Metric.wrl"
       (offset (xyz 0 0 0))
@@
   )
   (footprint "SamacSys_Parts:NHD0420AZFLYBW33V3" (layer "F.Cu")
-    (at 86.36 59.838)
+    (at 90.424 64.77)
     (descr "NHD-0420AZ-FL-YBW-33V3-2")
     (tags "Display")
@@
       (stroke (width 0.2) (type solid)) (layer "F.Fab"))
     (pad "1" thru_hole rect (at 0 0) (size 1.5 1.5) (drill 1) (layers "*.Cu" "*.Mask")
-      (net 30 "unconnected-(DS1-VSS-Pad1)") (pinfunction "VSS") (pintype "passive"))
+      (net 15 "+5V") (pinfunction "VSS") (pintype "passive"))
     (pad "2" thru_hole circle (at 2.54 0) (size 1.5 1.5) (drill 1) (layers "*.Cu" "*.Mask")
-      (net 31 "unconnected-(DS1-VDD-Pad2)") (pinfunction "VDD") (pintype "passive"))
+      (net 26 "GND") (pinfunction "VDD") (pintype "passive"))
     (pad "3" thru_hole circle (at 5.08 0) (size 1.5 1.5) (drill 1) (layers "*.Cu" "*.Mask")
       (net 37 "unconnected-(DS1-V0-Pad3)") (pinfunction "V0") (pintype "passive"))
@@
       (net 40 "unconnected-(DS1-E-Pad6)") (pinfunction "E") (pintype "passive"))
     (pad "7" thru_hole circle (at 15.24 0) (size 1.5 1.5) (drill 1) (layers "*.Cu" "*.Mask")
-      (net 41 "unconnected-(DS1-DB0-Pad7)") (pinfunction "DB0") (pintype "passive"))
+      (net 30 "Net-(DS1-DB0)") (pinfunction "DB0") (pintype "passive"))
     (pad "8" thru_hole circle (at 17.78 0) (size 1.5 1.5) (drill 1) (layers "*.Cu" "*.Mask")
-      (net 42 "unconnected-(DS1-DB1-Pad8)") (pinfunction "DB1") (pintype "passive"))
+      (net 31 "Net-(DS1-DB1)") (pinfunction "DB1") (pintype "passive"))
     (pad "9" thru_hole circle (at 20.32 0) (size 1.5 1.5) (drill 1) (layers "*.Cu" "*.Mask")
-      (net 43 "unconnected-(DS1-DB2-Pad9)") (pinfunction "DB2") (pintype "passive"))
+      (net 41 "Net-(DS1-DB2)") (pinfunction "DB2") (pintype "passive"))
     (pad "10" thru_hole circle (at 22.86 0) (size 1.5 1.5) (drill 1) (layers "*.Cu" "*.Mask")
-      (net 44 "unconnected-(DS1-DB3-Pad10)") (pinfunction "DB3") (pintype "passive"))
+      (net 42 "Net-(DS1-DB3)") (pinfunction "DB3") (pintype "passive"))
     (pad "11" thru_hole circle (at 25.4 0) (size 1.5 1.5) (drill 1) (layers "*.Cu" "*.Mask")
-      (net 45 "unconnected-(DS1-DB4-Pad11)") (pinfunction "DB4") (pintype "passive"))
+      (net 43 "Net-(DS1-DB4)") (pinfunction "DB4") (pintype "passive"))
     (pad "12" thru_hole circle (at 27.94 0) (size 1.5 1.5) (drill 1) (layers "*.Cu" "*.Mask")
-      (net 46 "unconnected-(DS1-DB5-Pad12)") (pinfunction "DB5") (pintype "passive"))
+      (net 44 "Net-(DS1-DB5)") (pinfunction "DB5") (pintype "passive"))
     (pad "13" thru_hole circle (at 30.48 0) (size 1.5 1.5) (drill 1) (layers "*.Cu" "*.Mask")
-      (net 47 "unconnected-(DS1-DB6-Pad13)") (pinfunction "DB6") (pintype "passive"))
+      (net 45 "Net-(DS1-DB6)") (pinfunction "DB6") (pintype "passive"))
     (pad "14" thru_hole circle (at 33.02 0) (size 1.5 1.5) (drill 1) (layers "*.Cu" "*.Mask")
-      (net 48 "unconnected-(DS1-DB7-Pad14)") (pinfunction "DB7") (pintype "passive"))
+      (net 46 "Net-(DS1-DB7)") (pinfunction "DB7") (pintype "passive"))
     (pad "15" thru_hole circle (at 35.56 0) (size 1.5 1.5) (drill 1) (layers "*.Cu" "*.Mask")
       (net 49 "unconnected-(DS1-LED+-Pad15)") (pinfunction "LED+") (pintype "passive"))
@@
       (net 50 "unconnected-(DS1-LED--Pad16)") (pinfunction "LED-") (pintype "passive"))
     (pad "MH1" thru_hole circle (at -6.5 1) (size 6 6) (drill 4) (layers "*.Cu" "*.Mask")
-      (net 51 "unconnected-(DS1-PadMH1)") (pinfunction "MH1") (pintype "passive"))
+      (net 26 "GND") (pinfunction "MH1") (pintype "passive"))
     (pad "MH2" thru_hole circle (at -6.5 41) (size 6 6) (drill 4) (layers "*.Cu" "*.Mask")
-      (net 52 "unconnected-(DS1-PadMH2)") (pinfunction "MH2") (pintype "passive"))
+      (net 26 "GND") (pinfunction "MH2") (pintype "passive"))
     (pad "MH3" thru_hole circle (at 63.5 41) (size 6 6) (drill 4) (layers "*.Cu" "*.Mask")
-      (net 53 "unconnected-(DS1-PadMH3)") (pinfunction "MH3") (pintype "passive"))
+      (net 26 "GND") (pinfunction "MH3") (pintype "passive"))
     (pad "MH4" thru_hole circle (at 63.5 1) (size 6 6) (drill 4) (layers "*.Cu" "*.Mask")
-      (net 54 "unconnected-(DS1-PadMH4)") (pinfunction "MH4") (pintype "passive"))
+      (net 26 "GND") (pinfunction "MH4") (pintype "passive"))
     (model "C:\\Users\\homer.morrill\\Documents\\KiCad\\SamacSys_Parts.3dshapes\\NHD-0420AZ-FL-YBW-33V3.stp"
       (offset (xyz 0 0 0))
@@
   (gr_circle (center 73 117) (end 72 116)
     (stroke (width 0.1) (type default)) (fill none) (layer "Edge.Cuts"))
-  (gr_circle (center 187 53) (end 186 52)
+  (gr_circle (center 187 53) (end 188.414214 53)
     (stroke (width 0.1) (type default)) (fill none) (layer "Edge.Cuts"))
   (gr_rect (start 70 50) (end 190 120)

Commit message: Update
Parts:
- added J3: Conn_01x03_Socket, Connector_JST:JST_EH_B3B-EH-A_1x03_P2.50mm_Vertical, F.Cu at (165.7, 112.2)
- added J4: AudioPlug3, Connector_Audio:Jack_3.5mm_Lumberg_1503_07_Horizontal, F.Cu at (165.4, 54.8)
- added U2: PCF8574, Package_DIP:DIP-8_W7.62mm, F.Cu at (170.4, 73.1)
- moved R1 67.8 mm to (137.2, 75.8)
Connections:
- U1 pad 22: unconnected-(U1-EXTCLK/PA0-Pad22) -> Net-(U1-EXTCLK/PA0)
Routing:
- net Net-(Q2-G): track 0.00 -> 17.2 mm
- net Net-(Q1-G): track 0.00 -> 15.7 mm
- net +5V: track 0.00 -> 13.1 mm
- net Net-(D2-A): track 0.00 -> 12.4 mm
- net Net-(D1-A): track 0.00 -> 10.5 mm
- net Net-(U1-UPDI): track 0.00 -> 4.39 mm
- added copper zone on B.Cu, net GND
- added copper zone on F.Cu, net GND

Commit message: Update
Parts:
- K1, K2: value Relay_SPDT -> AWHSH105D00G; footprint Relay_THT:Relay_SPST_Omron-G5Q-1A -> SamacSys_Parts:AWHSH105D00G
- moved K2 5.03 mm to (88.7, 100.4)
- moved K1 4.90 mm to (88.7, 81.9)
- renumbered Q2 to Q1, Q1 to Q2
Connections:
- K1 pad 1: (no net) -> Net-(D1-K)
- K1 pad 2: (no net) -> unconnected-(K1-NO-Pad2)
- K1 pad 3: (no net) -> unconnected-(K1-COIL_2-Pad3)
- K2 pad 1: (no net) -> Net-(D2-K)
- K2 pad 2: (no net) -> unconnected-(K2-NO-Pad2)
- K2 pad 3: (no net) -> unconnected-(K2-COIL_2-Pad3)
- U1 pad 14: unconnected-(U1-AVDD-Pad14) -> Net-(J3-Pin_1)
Routing:
- net +5V: track 13.1 -> 129.2 mm
- net Net-(DS1-DB3): track 0.00 -> 67.5 mm
- net Net-(DS1-DB1): track 0.00 -> 67.5 mm
- net Net-(DS1-DB2): track 0.00 -> 67.5 mm
- net Net-(DS1-DB0): track 0.00 -> 60.5 mm
- net Net-(J3-Pin_3): track 0.00 -> 51.2 mm, vias 0 -> 1
- net Net-(J3-Pin_1): track 0.00 -> 46.4 mm, vias 0 -> 2
- net Net-(J2-Pin_3): track 0.00 -> 46.2 mm
- net Net-(U1-EXTCLK/PA0): track 0.00 -> 44.6 mm, vias 0 -> 1
- net Net-(J2-Pin_4): track 0.00 -> 44.6 mm
- net Net-(J2-Pin_5): track 0.00 -> 42.9 mm
- net Net-(D1-K): track 0.00 -> 27.5 mm
- net Net-(D2-K): track 0.00 -> 25.9 mm
