File: 7.0/projects/BrevIce PCBA/BrevIce PCBA/BrevIce PCBA.kicad_sch (KiCad schematic)
At the start: 9 parts, among them J1 Conn_01x04_Socket, J2 Conn_01x05_Socket, K1 Relay_SPDT, K2 Relay_SPDT, Q1 AO3400A, Q2 AO3400A, U1 ATmega3208-X

Commit message: Update BrevIce PCBA.kicad_sch
Parts:
- added DS1: NHD-0420AZ-FL-YBW-33V3, SamacSys_Parts:NHD0420AZFLYBW33V3, symbol SamacSys_Parts:NHD-0420AZ-FL-YBW-33V3
- added J3: Conn_01x03_Socket, symbol Connector:Conn_01x03_Socket
- added R1: 4.7K, Resistor_SMD:R_0603_1608Metric_Pad0.98x0.95mm_HandSolder, symbol Device:R_Small
Connections:
- net GND: now also J3.2 (Pin_2)
- net at U1.19 (UPDI): now also R1.1
- net at U1.20 (VDD): now also J3.1 (Pin_1)
- new net: J3.3 (Pin_3), R1.2
Changed lines of the file:
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@@
+    (stroke (width 0) (type default))
+  )
+  (wire (pts (xy 50.8 36.83) (xy 76.2 36.83))
     (stroke (width 0) (type default))
   )
@@
     (stroke (width 0) (type default))
   )
+  (wire (pts (xy 81.28 36.83) (xy 86.36 36.83))
+    (stroke (width 0) (type default))
+  )
   (wire (pts (xy 128.27 80.01) (xy 138.43 80.01))
     (stroke (width 0) (type default))
@@
     (stroke (width 0) (type default))
   )
+  (wire (pts (xy 50.8 33.02) (xy 72.39 33.02))
+    (stroke (width 0) (type default))
+  )
   (wire (pts (xy 160.02 102.87) (xy 160.02 107.95))
     (stroke (width 0) (type default))
@@
     (stroke (width 0) (type default))
   )
+  (wire (pts (xy 50.8 30.48) (xy 101.6 30.48))
+    (stroke (width 0) (type default))
+  )
+  (wire (pts (xy 101.6 31.75) (xy 101.6 30.48))
+    (stroke (width 0) (type default))
+  )
   (wire (pts (xy 116.84 46.99) (xy 156.21 46.99))
     (stroke (width 0) (type default))
   )
+  (wire (pts (xy 72.39 27.94) (xy 72.39 33.02))
+    (stroke (width 0) (type default))
+  )
   (wire (pts (xy 116.84 64.77) (xy 124.46 64.77))
     (stroke (width 0) (type default))
@@
     (stroke (width 0) (type default))
   )
+  (wire (pts (xy 50.8 36.83) (xy 50.8 35.56))
+    (stroke (width 0) (type default))
+  )
   (wire (pts (xy 52.07 74.93) (xy 86.36 74.93))
     (stroke (width 0) (type default))
@@
   (wire (pts (xy 116.84 59.69) (xy 128.27 59.69))
     (stroke (width 0) (type default))
+  )
+  (symbol (lib_id "power:GND") (at 72.39 27.94 0) (mirror x) (unit 1)
+    (in_bom yes) (on_board yes) (dnp no)
+    (property "Reference" "#PWR01" (at 72.39 21.59 0)
+      (effects (font (size 1.27 1.27)) hide)
+    )
+    (property "Value" "GND" (at 72.39 22.86 0)
+      (effects (font (size 1.27 1.27)))
+    )
+    (property "Footprint" "" (at 72.39 27.94 0)
+      (effects (font (size 1.27 1.27)) hide)
+    )
+    (property "Datasheet" "" (at 72.39 27.94 0)
+      (effects (font (size 1.27 1.27)) hide)
+    )
+    (pin "1")
+    (instances
+      (project "BrevIce PCBA"
+        (path "/eebd9bfd-78a7-4078-9512-a76ab1c9463f"
+          (reference "#PWR01") (unit 1)
+        )
+      )
+    )
   )
   (symbol (lib_id "power:GND") (at 101.6 87.63 0) (unit 1)
@@
         (path "/eebd9bfd-78a7-4078-9512-a76ab1c9463f"
           (reference "D2") (unit 1)
+        )
+      )
+    )
+  )
+  (symbol (lib_id "SamacSys_Parts:NHD-0420AZ-FL-YBW-33V3") (at 76.2 133.35 0) (unit 1)
+    (in_bom yes) (on_board yes) (dnp no) (fields_autoplaced)
+    (property "Reference" "DS1" (at 90.17 125.73 0)
+      (effects (font (size 1.27 1.27)))
+    )
+    (property "Value" "NHD-0420AZ-FL-YBW-33V3" (at 90.17 128.27 0)
+      (effects (font (size 1.27 1.27)))
+    )
+    (property "Footprint" "SamacSys_Parts:NHD0420AZFLYBW33V3" (at 100.33 130.81 0)
+      (effects (font (size 1.27 1.27)) (justify left) hide)
+    )
+    (property "Datasheet" "https://www.newhavendisplay.com/specs/NHD-0420AZ-FL-YBW-33V3.pdf" (at 100.33 133.35 0)
+      (effects (font (size 1.27 1.27)) (justify left) hide)
+    )
+    (property "Description" "LCD Character Display Modules & Accessories STN-Y/G Transfl 77.5 x 47.0" (at 100.33 135.89 0)
+      (effects (font (size 1.27 1.27)) (justify left) hide)
+    )
+    (property "Height" "14.5" (at 100.33 138.43 0)
+      (effects (font (size 1.27 1.27)) (justify left) hide)
+    )
+    (property "Mouser Part Number" "763-0420AZFLYBW33V3" (at 100.33 140.97 0)
+      (effects (font (size 1.27 1.27)) (justify left) hide)
+    )
+    (property "Mouser Price/Stock" "https://www.mouser.co.uk/ProductDetail/Newhaven-Display/NHD-0420AZ-FL-YBW-33V3?qs=G49gCGQm93hSVvgE4zZg6g%3D%3D" (at 100.33 143.51 0)
+      (effects (font (size 1.27 1.27)) (justify left) hide)
+    )
+    (property "Manufacturer_Name" "Newhaven Display" (at 100.33 146.05 0)
+      (effects (font (size 1.27 1.27)) (justify left) hide)
+    )
+    (property "Manufacturer_Part_Number" "NHD-0420AZ-FL-YBW-33V3" (at 100.33 148.59 0)
+      (effects (font (size 1.27 1.27)) (justify left) hide)
+    )
+    (pin "1")
+    (pin "10")
+    (pin "11")
+    (pin "12")
+    (pin "13")
+    (pin "14")
+    (pin "15")
+    (pin "16")
+    (pin "2")
+    (pin "3")
+    (pin "4")
+    (pin "5")
+    (pin "6")
+    (pin "7")
+    (pin "8")
+    (pin "9")
+    (pin "MH1")
+    (pin "MH2")
+    (pin "MH3")
+    (pin "MH4")
+    (instances
+      (project "BrevIce PCBA"
+        (path "/eebd9bfd-78a7-4078-9512-a76ab1c9463f"
+          (reference "DS1") (unit 1)
         )
       )
@@
     )
   )
+  (symbol (lib_id "Connector:Conn_01x03_Socket") (at 45.72 33.02 0) (mirror y) (unit 1)
+    (in_bom yes) (on_board yes) (dnp no)
+    (property "Reference" "J3" (at 44.45 31.75 0)
+      (effects (font (size 1.27 1.27)) (justify left))
+    )
+    (property "Value" "Conn_01x03_Socket" (at 44.45 34.29 0)
+      (effects (font (size 1.27 1.27)) (justify left))
+    )
+    (property "Footprint" "" (at 45.72 33.02 0)
+      (effects (font (size 1.27 1.27)) hide)
+    )
+    (property "Datasheet" "~" (at 45.72 33.02 0)
+      (effects (font (size 1.27 1.27)) hide)
+    )
+    (pin "1")
+    (pin "2")
+    (pin "3")
+    (instances
+      (project "BrevIce PCBA"
+        (path "/eebd9bfd-78a7-4078-9512-a76ab1c9463f"
+          (reference "J3") (unit 1)
+        )
+      )
+    )
+  )
   (symbol (lib_id "Connector:Conn_01x04_Socket") (at 161.29 46.99 0) (unit 1)
     (in_bom yes) (on_board yes) (dnp no) (fields_autoplaced)
@@
         )
       )
+    )
+  )
+  (symbol (lib_id "Device:R_Small") (at 78.74 36.83 270) (unit 1)
+    (in_bom yes) (on_board yes) (dnp no) (fields_autoplaced)
+    (property "Reference" "R1" (at 78.74 31.75 90)
+      (effects (font (size 1.27 1.27)))
+    )
+    (property "Value" "4.7K" (at 78.74 34.29 90)
+      (effects (font (size 1.27 1.27)))
+    )
+    (property "Footprint" "Resistor_SMD:R_0603_1608Metric_Pad0.98x0.95mm_HandSolder" (at 78.74 36.83 0)
+      (effects (font (size 1.27 1.27)) hide)
+    )
+    (property "Datasheet" "~" (at 78.74 36.83 0)
+      (effects (font (size 1.27 1.27)) hide)
+    )
+    (pin "1")
+    (pin "2")
+    (instances
+      (project "BrevIce PCBA"
+        (path "/eebd9bfd-78a7-4078-9512-a76ab1c9463f"
+          (reference "R1") (unit 1)
+        )
+      )

Commit message: Update
Parts:
- added U2: PCF8574, symbol Interface_Expansion:PCF8574
Connections:
- net +5V: now also DS1.1 (VSS), U2.8 (VSS)
- net GND: now also DS1.2 (VDD), DS1.MH1, DS1.MH2, DS1.MH3, DS1.MH4, U2.16 (VDD)
- net at DS1.10 (DB3): now also U2.7 (P3)
- net at DS1.11 (DB4): now also U2.9 (P4)
- net at DS1.12 (DB5): now also U2.10 (P5)
- net at DS1.13 (DB6): now also U2.11 (P6)
- net at DS1.14 (DB7): now also U2.12 (P7)
- net at DS1.7 (DB0): now also U2.4 (P0)
- net at DS1.8 (DB1): now also U2.5 (P1)
- net at DS1.9 (DB2): now also U2.6 (P2)
Other:
- moved on the sheet: D1, D2, DS1, K1, K2, Q1, Q2

Commit message: Update
Parts:
- removed J1: Conn_01x04_Socket, Connector_JST:JST_EH_B4B-EH-A_1x04_P2.50mm_Vertical, symbol Connector:Conn_01x04_Socket
Connections:
- net at U2.14 (SCL): now also U1.25 (PA3)
- net at U2.15 (SDA): now also U1.24 (PA2)
Changed lines of the file:
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@@
+    (stroke (width 0) (type default))
+  )
+  (wire (pts (xy 116.84 49.53) (xy 129.54 49.53))
     (stroke (width 0) (type default))
   )
@@
     (stroke (width 0) (type default))
   )
+  (wire (pts (xy 102.87 99.06) (xy 102.87 102.87))
+    (stroke (width 0) (type default))
+  )
+  (wire (pts (xy 116.84 46.99) (xy 132.08 46.99))
+    (stroke (width 0) (type default))
+  )
+  (wire (pts (xy 100.33 96.52) (xy 100.33 102.87))
+    (stroke (width 0) (type default))
+  )
   (wire (pts (xy 110.49 135.89) (xy 128.27 135.89))
     (stroke (width 0) (type default))
@@
     (stroke (width 0) (type default))
   )
-  (wire (pts (xy 116.84 49.53) (xy 156.21 49.53))
-    (stroke (width 0) (type default))
-  )
   (wire (pts (xy 125.73 160.02) (xy 135.89 160.02))
     (stroke (width 0) (type default))
@@
     (stroke (width 0) (type default))
   )
+  (wire (pts (xy 129.54 96.52) (xy 100.33 96.52))
+    (stroke (width 0) (type default))
+  )
   (wire (pts (xy 128.27 135.89) (xy 128.27 152.4))
     (stroke (width 0) (type default))
@@
     (stroke (width 0) (type default))
   )
-  (wire (pts (xy 116.84 46.99) (xy 156.21 46.99))
-    (stroke (width 0) (type default))
-  )
   (wire (pts (xy 107.95 128.27) (xy 107.95 135.89))
     (stroke (width 0) (type default))
@@
     (stroke (width 0) (type default))
   )
+  (wire (pts (xy 132.08 46.99) (xy 132.08 99.06))
+    (stroke (width 0) (type default))
+  )
   (wire (pts (xy 72.39 27.94) (xy 72.39 33.02))
     (stroke (width 0) (type default))
@@
     (stroke (width 0) (type default))
   )
+  (wire (pts (xy 132.08 99.06) (xy 102.87 99.06))
+    (stroke (width 0) (type default))
+  )
   (wire (pts (xy 100.33 128.27) (xy 72.39 128.27))
     (stroke (width 0) (type default))
@@
   )
   (wire (pts (xy 133.35 130.81) (xy 133.35 157.48))
+    (stroke (width 0) (type default))
+  )
+  (wire (pts (xy 129.54 49.53) (xy 129.54 96.52))
     (stroke (width 0) (type default))
   )
@@
         )
       )
-    )
-  )
-  (symbol (lib_id "Connector:Conn_01x04_Socket") (at 161.29 46.99 0) (unit 1)
-    (in_bom yes) (on_board yes) (dnp no) (fields_autoplaced)
-    (property "Reference" "J1" (at 162.56 46.99 0)
-      (effects (font (size 1.27 1.27)) (justify left))
-    )
-    (property "Value" "Conn_01x04_Socket" (at 162.56 49.53 0)
-      (effects (font (size 1.27 1.27)) (justify left))
-    )
-    (property "Footprint" "Connector_JST:JST_EH_B4B-EH-A_1x04_P2.50mm_Vertical" (at 161.29 46.99 0)
-      (effects (font (size 1.27 1.27)) hide)
-    )
-    (property "Datasheet" "~" (at 161.29 46.99 0)
-      (effects (font (size 1.27 1.27)) hide)
-    )
-    (pin "1")
-    (pin "2")
-    (pin "3")
-    (pin "4")
-    (instances
-      (project "BrevIce PCBA"
-        (path "/eebd9bfd-78a7-4078-9512-a76ab1c9463f"
-          (reference "J1") (unit 1)
-        )
-      )

Commit message: Update
Connections:
- net +5V: now also U2.16 (VDD); no longer U2.8 (VSS)
- net GND: now also U2.8 (VSS); no longer U2.16 (VDD)
Changed lines of the file:
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@@
     (stroke (width 0) (type default))
+  )
+  (symbol (lib_id "power:+5V") (at 90.17 115.57 0) (mirror x) (unit 1)
+    (in_bom yes) (on_board yes) (dnp no)
+    (property "Reference" "#PWR09" (at 90.17 111.76 0)
+      (effects (font (size 1.27 1.27)) hide)
+    )
+    (property "Value" "+5V" (at 90.17 120.65 0)
+      (effects (font (size 1.27 1.27)))
+    )
+    (property "Footprint" "" (at 90.17 115.57 0)
+      (effects (font (size 1.27 1.27)) hide)
+    )
+    (property "Datasheet" "" (at 90.17 115.57 0)
+      (effects (font (size 1.27 1.27)) hide)
+    )
+    (pin "1")
+    (instances
+      (project "BrevIce PCBA"
+        (path "/eebd9bfd-78a7-4078-9512-a76ab1c9463f"
+          (reference "#PWR09") (unit 1)
+        )
+      )
+    )
   )
   (symbol (lib_id "power:GND") (at 72.39 27.94 0) (mirror x) (unit 1)
@@
         (path "/eebd9bfd-78a7-4078-9512-a76ab1c9463f"
           (reference "U2") (unit 1)
+        )
+      )
+    )
+  )
+  (symbol (lib_id "power:GND") (at 132.08 115.57 0) (unit 1)
+    (in_bom yes) (on_board yes) (dnp no) (fields_autoplaced)
+    (property "Reference" "#PWR010" (at 132.08 121.92 0)
+      (effects (font (size 1.27 1.27)) hide)
+    )
+    (property "Value" "GND" (at 132.08 120.65 0)
+      (effects (font (size 1.27 1.27)))
+    )
+    (property "Footprint" "" (at 132.08 115.57 0)
+      (effects (font (size 1.27 1.27)) hide)
+    )
+    (property "Datasheet" "" (at 132.08 115.57 0)
+      (effects (font (size 1.27 1.27)) hide)
+    )
+    (pin "1")
+    (instances
+      (project "BrevIce PCBA"
+        (path "/eebd9bfd-78a7-4078-9512-a76ab1c9463f"
+          (reference "#PWR010") (unit 1)
         )
       )
@@
     )
   )
-  (symbol (lib_id "power:GND") (at 90.17 115.57 0) (unit 1)
-    (in_bom yes) (on_board yes) (dnp no) (fields_autoplaced)
-    (property "Reference" "#PWR010" (at 90.17 121.92 0)
-      (effects (font (size 1.27 1.27)) hide)
-    )
-    (property "Value" "GND" (at 90.17 120.65 0)
-      (effects (font (size 1.27 1.27)))
-    )
-    (property "Footprint" "" (at 90.17 115.57 0)
-      (effects (font (size 1.27 1.27)) hide)
-    )
-    (property "Datasheet" "" (at 90.17 115.57 0)
-      (effects (font (size 1.27 1.27)) hide)
-    )
-    (pin "1")
-    (instances
-      (project "BrevIce PCBA"
-        (path "/eebd9bfd-78a7-4078-9512-a76ab1c9463f"
-          (reference "#PWR010") (unit 1)
-        )
-      )
-    )
-  )
   (symbol (lib_id "power:GND") (at 226.06 106.68 0) (unit 1)
     (in_bom yes) (on_board yes) (dnp no) (fields_autoplaced)
@@
         )
       )
-    )
-  )
-  (symbol (lib_id "power:+5V") (at 132.08 115.57 0) (unit 1)
-    (in_bom yes) (on_board yes) (dnp no) (fields_autoplaced)
-    (property "Reference" "#PWR09" (at 132.08 119.38 0)
-      (effects (font (size 1.27 1.27)) hide)
-    )
-    (property "Value" "+5V" (at 132.08 110.49 0)
-      (effects (font (size 1.27 1.27)))
-    )
-    (property "Footprint" "" (at 132.08 115.57 0)
-      (effects (font (size 1.27 1.27)) hide)
-    )
-    (property "Datasheet" "" (at 132.08 115.57 0)
-      (effects (font (size 1.27 1.27)) hide)
-    )
-    (pin "1")
-    (instances
-      (project "BrevIce PCBA"
-        (path "/eebd9bfd-78a7-4078-9512-a76ab1c9463f"
-          (reference "#PWR09") (unit 1)
-        )
-      )

Commit message: Update
Parts:
- added J4: AudioPlug3, Connector_Audio:Jack_3.5mm_Lumberg_1503_07_Horizontal, symbol Connector_Audio:AudioPlug3
- J3: footprint (none) -> Connector_JST:JST_EH_B3B-EH-A_1x03_P2.50mm_Vertical
- U2: footprint (none) -> Package_DIP:DIP-8_W7.62mm
Connections:
- net +5V: now also J4.S
- net GND: now also J4.T
- net at U1.22 (EXTCLK/PA0): now also J4.R
Changed lines of the file:
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@@
+    (stroke (width 0) (type default))
+  )
+  (wire (pts (xy 127 30.48) (xy 127 41.91))
     (stroke (width 0) (type default))
   )
@@
     (stroke (width 0) (type default))
   )
+  (wire (pts (xy 151.13 30.48) (xy 127 30.48))
+    (stroke (width 0) (type default))
+  )
   (wire (pts (xy 110.49 135.89) (xy 128.27 135.89))
     (stroke (width 0) (type default))
@@
     (stroke (width 0) (type default))
   )
+  (wire (pts (xy 127 41.91) (xy 116.84 41.91))
+    (stroke (width 0) (type default))
+  )
   (wire (pts (xy 80.01 175.26) (xy 97.79 175.26))
     (stroke (width 0) (type default))
@@
     (stroke (width 0) (type default))
   )
+  (wire (pts (xy 151.13 33.02) (xy 151.13 35.56))
+    (stroke (width 0) (type default))
+  )
   (wire (pts (xy 77.47 133.35) (xy 77.47 172.72))
     (stroke (width 0) (type default))
@@
   )
   (wire (pts (xy 113.03 128.27) (xy 113.03 133.35))
+    (stroke (width 0) (type default))
+  )
+  (wire (pts (xy 151.13 22.86) (xy 151.13 27.94))
     (stroke (width 0) (type default))
   )
@@
       (effects (font (size 1.27 1.27)))
     )
-    (property "Footprint" "" (at 110.49 115.57 0)
+    (property "Footprint" "Package_DIP:DIP-8_W7.62mm" (at 110.49 115.57 0)
       (effects (font (size 1.27 1.27)) hide)
     )
@@
     )
   )
+  (symbol (lib_id "power:GND") (at 151.13 35.56 0) (unit 1)
+    (in_bom yes) (on_board yes) (dnp no) (fields_autoplaced)
+    (property "Reference" "#PWR012" (at 151.13 41.91 0)
+      (effects (font (size 1.27 1.27)) hide)
+    )
+    (property "Value" "GND" (at 151.13 40.64 0)
+      (effects (font (size 1.27 1.27)))
+    )
+    (property "Footprint" "" (at 151.13 35.56 0)
+      (effects (font (size 1.27 1.27)) hide)
+    )
+    (property "Datasheet" "" (at 151.13 35.56 0)
+      (effects (font (size 1.27 1.27)) hide)
+    )
+    (pin "1")
+    (instances
+      (project "BrevIce PCBA"
+        (path "/eebd9bfd-78a7-4078-9512-a76ab1c9463f"
+          (reference "#PWR012") (unit 1)
+        )
+      )
+    )
+  )
   (symbol (lib_id "Connector:Conn_01x03_Socket") (at 45.72 33.02 0) (mirror y) (unit 1)
     (in_bom yes) (on_board yes) (dnp no)
@@
       (effects (font (size 1.27 1.27)) (justify left))
     )
-    (property "Footprint" "" (at 45.72 33.02 0)
+    (property "Footprint" "Connector_JST:JST_EH_B3B-EH-A_1x03_P2.50mm_Vertical" (at 45.72 33.02 0)
       (effects (font (size 1.27 1.27)) hide)
     )
@@
         (path "/eebd9bfd-78a7-4078-9512-a76ab1c9463f"
           (reference "#PWR02") (unit 1)
+        )
+      )
+    )
+  )
+  (symbol (lib_id "power:+5V") (at 151.13 22.86 0) (mirror y) (unit 1)
+    (in_bom yes) (on_board yes) (dnp no)
+    (property "Reference" "#PWR013" (at 151.13 26.67 0)
+      (effects (font (size 1.27 1.27)) hide)
+    )
+    (property "Value" "+5V" (at 151.13 17.78 0)
+      (effects (font (size 1.27 1.27)))
+    )
+    (property "Footprint" "" (at 151.13 22.86 0)
+      (effects (font (size 1.27 1.27)) hide)
+    )
+    (property "Datasheet" "" (at 151.13 22.86 0)
+      (effects (font (size 1.27 1.27)) hide)
+    )
+    (pin "1")
+    (instances
+      (project "BrevIce PCBA"
+        (path "/eebd9bfd-78a7-4078-9512-a76ab1c9463f"
+          (reference "#PWR013") (unit 1)
         )
       )
@@
         )
       )
+    )
+  )
+  (symbol (lib_id "Connector_Audio:AudioPlug3") (at 166.37 30.48 0) (mirror y) (unit 1)
+    (in_bom yes) (on_board yes) (dnp no)
+    (property "Reference" "J4" (at 166.37 20.32 0)
+      (effects (font (size 1.27 1.27)))
+    )
+    (property "Value" "AudioPlug3" (at 166.37 22.86 0)
+      (effects (font (size 1.27 1.27)))
+    )
+    (property "Footprint" "Connector_Audio:Jack_3.5mm_Lumberg_1503_07_Horizontal" (at 163.83 31.75 0)
+      (effects (font (size 1.27 1.27)) hide)
+    )
+    (property "Datasheet" "~" (at 163.83 31.75 0)
+      (effects (font (size 1.27 1.27)) hide)
+    )
+    (pin "R")
+    (pin "S")
+    (pin "T")
+    (instances
+      (project "BrevIce PCBA"
+        (path "/eebd9bfd-78a7-4078-9512-a76ab1c9463f"
+          (reference "J4") (unit 1)
+        )
+      )

Commit message: Update
Parts:
- removed K1, K2: Relay_SPDT, Relay_THT:Relay_SPST_Omron-G5Q-1A, symbol Relay:Relay_SPDT
- added K1, K2: AWHSH105D00G, AWHSH105D00G, symbol SamacSys_Parts:AWHSH105D00G
- renumbered Q2 to Q1, Q1 to Q2
Connections:
- net GND: now also K1.4 (COM), K2.4 (COM)
- net at D2.1 (K): now also K2.1 (COIL_1)
- net at J3.1 (Pin_1), U1.20 (VDD): now also U1.14 (AVDD)
- net at D1.1 (K): now also K1.1 (COIL_1)
- no-connect marks 2 -> 0
