File: 7.0/projects/Batt_Pack/Batt_Pack/Batt_Pack.kicad_sch (KiCad schematic)
At the start: 2 parts, among them U2 ATmega3208-X

Commit message: Update
Parts:
- U1: footprint (none) -> Package_QFP:TQFP-64_10x10mm_P0.5mm
Changed lines of the file:
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@@
       (effects (font (size 1.27 1.27)))
     )
-    (property "Footprint" "" (at 138.43 96.52 0)
+    (property "Footprint" "Package_QFP:TQFP-64_10x10mm_P0.5mm" (at 138.43 96.52 0)
       (effects (font (size 1.27 1.27)) hide)
     )
