File: 7.0/projects/Control Pilot PCB AUTO/Control Pilot PCB/Control Pilot PCB.kicad_pcb (KiCad board)
At the start: 2 copper layers, 125 x 75 mm, 25 parts, among them J1 Conn_01x01, J2 Conn_01x01, J3 Conn_01x01, J4 Conn_01x01, J5 Conn_01x01, Q1 AO3400A, Q2 AO3400A, SW1 SW_SPDT, SW2 SW_SPDT, SW3 SW_SPDT, SW5 SW_SPDT, SW6 SW_SPDT, SW7 SW_SPDT

Commit message: Update
Parts:
- removed SW7: SW_SPDT, Connector_PinHeader_2.54mm:PinHeader_1x03_P2.54mm_Vertical
- added SW4: SW_SPDT, Connector_PinHeader_2.54mm:PinHeader_1x03_P2.54mm_Vertical, F.Cu at (118.4, 82.0)
- C1: value C_Polarized -> 100uF
- C2: value C_Polarized -> 200uF
- moved J5 173.3 mm to (271.2, 67.1), turned to 0 degrees
- moved Q1 163.3 mm to (246.0, 85.9), turned to 0 degrees
- moved J4 160.2 mm to (272.3, 75.7), turned to 0 degrees
- moved Q2 154.7 mm to (234.0, 87.2), turned to 0 degrees
- moved R1 136.5 mm to (207.4, 92.8), turned to 0 degrees
- moved C1 123.7 mm to (191.8, 37.8), turned to 0 degrees
- moved J1 122.4 mm to (271.4, 45.7), turned to 0 degrees
- moved R2 118.3 mm to (187.5, 53.0), turned to 0 degrees
- moved R9 116.2 mm to (190.0, 91.3), turned to 0 degrees
- moved R8 115.6 mm to (190.0, 83.0), turned to 0 degrees
- moved J2 109.3 mm to (272.9, 85.9), turned to 0 degrees
- moved J3 108.7 mm to (271.3, 55.3), turned to 0 degrees
- moved R3 89.8 mm to (187.5, 56.1), turned to 0 degrees
- moved C2 72.4 mm to (155.0, 60.3), turned to 0 degrees
- moved R4 64.3 mm to (187.5, 59.2), turned to 0 degrees
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Connections:
- Q1 pad 3: Net-(D1-K) -> Net-(Q1-D)
- Q2 pad 3: Net-(D1-K) -> Net-(Q1-D)
- R1 pad 1: Net-(SW1-A) -> Net-(D1-K)
- R2 pad 1: Net-(SW1-A) -> Net-(D1-K)
- R3 pad 1: Net-(SW1-A) -> Net-(SW4-B)
- R3 pad 2: Net-(SW7-B) -> Net-(D1-K)
- R7 pad 1: Net-(SW6-A) -> Net-(SW6-B)
- R8 pad 1: Net-(SW1-A) -> Net-(D1-K)
- R9 pad 1: Net-(SW1-A) -> Net-(D1-K)
- SW1 pad 1: Net-(SW1-A) -> Net-(Q1-D)
- SW2 pad 1: Net-(SW1-A) -> unconnected-(SW2-A-Pad1)
- SW2 pad 2: Net-(SW1-A) -> Net-(Q1-D)
- SW3 pad 1: Net-(SW1-A) -> unconnected-(SW3-A-Pad1)
- SW3 pad 2: Net-(SW1-A) -> Net-(Q1-D)
- SW6 pad 2: Earth_Protective -> Net-(SW6-B)
- SW6 pad 3: unconnected-(SW6-C-Pad3) -> Earth_Protective
Routing:
- net Earth_Protective: track 234.2 -> 0.00 mm
- net Net-(SW1-A): track 136.4 -> 0.00 mm
- net +5V: track 98.4 -> 0.00 mm
- net Net-(D1-K): track 82.8 -> 0.00 mm
- net Net-(D1-A): track 58.2 -> 0.00 mm
- net Net-(J3-Pin_1): track 35.0 -> 0.00 mm
- net Net-(SW5-A): track 22.6 -> 0.00 mm
- net Net-(Q2-S): track 20.7 -> 0.00 mm
- net Net-(Q1-S): track 18.9 -> 0.00 mm
- net Net-(SW6-A): track 16.8 -> 0.00 mm
- net Net-(SW7-B): track 9.11 -> 0.00 mm
- net Net-(C1-Pad1): track 7.60 -> 0.00 mm
- net Net-(C2-Pad1): track 7.48 -> 0.00 mm
- net Net-(Q2-G): track 6.73 -> 0.00 mm
- net Net-(Q1-G): track 5.13 -> 0.00 mm
Other:
- board text removed: "+5V-"
- board text removed: "D"
- board text removed: "E"
- board text removed: "F"
- board text removed: "GND-"
- board text removed: "PE"
- board text removed: "S1"
- board text removed: "S2"
