File: 7.0/projects/Control Pilot PCB/Control Pilot PCB/Control Pilot PCB ORIGINAL.kicad_pcb (KiCad board)
At the start: 2 copper layers, 125 x 75 mm, 21 parts, among them J1 Conn_01x01, J2 Conn_01x01, J3 Conn_01x01, J4 Conn_01x01, J5 Conn_01x01, SW1 SW_SPDT, SW2 SW_SPDT, SW3 SW_SPDT, SW4 SW_SPDT, SW5 SW_SPDT, SW6 SW_SPDT, SW7 SW_SPDT, SW8 SW_SPDT

Commit message: Mass Update
Routing:
- net Earth_Protective: track 197.5 -> 0.00 mm
Changed lines of the file:
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@@
     (effects (font (size 1.75 1.75) (thickness 0.4) bold) (justify left bottom mirror))
   )
-  (segment (start 167.64 96.52) (end 167.64 61.976) (width 0.4) (layer "F.Cu") (net 1))
-  (segment (start 167.64 61.976) (end 164.592 58.928) (width 0.4) (layer "F.Cu") (net 1))
-  (segment (start 143.256 101.092) (end 148.336 96.012) (width 0.4) (layer "F.Cu") (net 1))
-  (segment (start 98.552 54.864) (end 98.552 52.832) (width 0.4) (layer "F.Cu") (net 1))
-  (segment (start 163.576 101.092) (end 163.576 100.584) (width 0.4) (layer "F.Cu") (net 1))
-  (segment (start 149.844 82.804) (end 150.876 82.804) (width 0.4) (layer "F.Cu") (net 1))
-  (segment (start 143.256 101.092) (end 163.576 101.092) (width 0.4) (layer "F.Cu") (net 1))
-  (segment (start 163.576 103.632) (end 163.576 101.092) (width 0.4) (layer "F.Cu") (net 1))
-  (segment (start 164.084 93.472) (end 166.624 90.932) (width 0.4) (layer "F.Cu") (net 1))
-  (segment (start 144.256 88.392) (end 149.844 82.804) (width 0.4) (layer "F.Cu") (net 1))
-  (segment (start 163.576 100.584) (end 167.64 96.52) (width 0.4) (layer "F.Cu") (net 1))
-  (segment (start 164.592 58.928) (end 102.616 58.928) (width 0.4) (layer "F.Cu") (net 1))
-  (segment (start 156.972 93.472) (end 164.084 93.472) (width 0.4) (layer "F.Cu") (net 1))
-  (segment (start 166.624 83.82) (end 165.608 82.804) (width 0.4) (layer "F.Cu") (net 1))
-  (segment (start 148.336 96.012) (end 154.432 96.012) (width 0.4) (layer "F.Cu") (net 1))
-  (segment (start 166.624 90.932) (end 166.624 83.82) (width 0.4) (layer "F.Cu") (net 1))
-  (segment (start 154.432 96.012) (end 156.972 93.472) (width 0.4) (layer "F.Cu") (net 1))
-  (segment (start 165.608 82.804) (end 150.876 82.804) (width 0.4) (layer "F.Cu") (net 1))
-  (segment (start 102.616 58.928) (end 98.552 54.864) (width 0.4) (layer "F.Cu") (net 1))
   (segment (start 163.576 86.36) (end 150.876 86.36) (width 0.4) (layer "F.Cu") (net 2))
   (segment (start 119.616 98.552) (end 117.584 96.52) (width 0.4) (layer "F.Cu") (net 2))
