File: 7.0/projects/Control Pilot PCB/Control Pilot PCB/Control Pilot PCB.kicad_pcb (KiCad board)
At the start: 2 copper layers, 125 x 75 mm, 21 parts, among them J1 Conn_01x01, J2 Conn_01x01, J3 Conn_01x01, J4 Conn_01x01, J5 Conn_01x01, SW1 SW_SPDT, SW2 SW_SPDT, SW3 SW_SPDT, SW4 SW_SPDT, SW5 SW_SPDT, SW6 SW_SPDT, SW7 SW_SPDT, SW8 SW_SPDT

Commit message: Update
Routing:
- net Net-(D1-K): track 106.7 -> 107.2 mm

Commit message: Update
Connections:
- R1 pad 2: Net-(SW4-B) -> Net-(D1-K)
- SW4 pad 2: Net-(SW4-B) -> Net-(D1-K)
Routing:
- net Earth_Protective: track 197.5 -> 164.5 mm
- net Net-(D1-K): track 107.2 -> 117.5 mm
- net Net-(SW4-B): track 10.2 -> 0.00 mm
- net Net-(SW1-A): track 144.0 -> 146.3 mm
- added copper zone on B.Cu, net Earth_Protective
- added copper zone on F.Cu, net Earth_Protective

Commit message: update
Parts:
- SW1, SW2, SW3, SW4, SW5, SW6, SW7, SW8: moved to B.Cu
- moved SW1 76.2 mm to (67.1, 103.6), turned to 0 degrees
- moved SW4 76.2 mm to (143.3, 103.6), turned to 0 degrees
- moved SW5 76.2 mm to (67.1, 72.5), turned to 0 degrees
- moved SW8 76.2 mm to (143.3, 72.5), turned to 0 degrees
- moved SW2 28.9 mm to (90.7, 103.6), turned to 0 degrees
- moved SW3 25.4 mm to (117.9, 103.6), turned to 0 degrees
- moved SW6 25.4 mm to (92.5, 73.2), turned to 0 degrees
- moved SW7 25.4 mm to (117.9, 72.5), turned to 0 degrees
