File: 7.0/projects/Control Pilot PCB/Control Pilot PCB/Control Pilot PCB.kicad_sch (KiCad schematic)
At the start: 21 parts, among them J1 Conn_01x01, J2 Conn_01x01, J3 Conn_01x01, J4 Conn_01x01, J5 Conn_01x01, SW1 SW_SPDT, SW2 SW_SPDT, SW3 SW_SPDT, SW4 SW_SPDT, SW5 SW_SPDT, SW6 SW_SPDT, SW7 SW_SPDT, SW8 SW_SPDT

Commit message: Update
Other:
- company: (none) -> Power Innovations International
- title: (none) -> Control Pilot PCB
Changed lines of the file:
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@@
 (kicad_sch (version 20230121) (generator eeschema)
   (paper "A4")
+  (title_block
+    (title "Control Pilot PCB")
+    (date "12/14/2023")
+    (rev "1.0")
+    (company "Power Innovations International")
+    (comment 3 "Created By: Homer Morrill")
+  )
   (junction (at 231.14 74.93) (diameter 0) (color 0 0 0 0)
   )

Commit message: update
Changed lines of the file:
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@@
   (junction (at 231.14 52.07) (diameter 0) (color 0 0 0 0)
+  )
+  (junction (at 77.47 118.11) (diameter 0) (color 0 0 0 0)
   )
   (junction (at 168.91 52.07) (diameter 0) (color 0 0 0 0)
@@
   (junction (at 189.23 99.06) (diameter 0) (color 0 0 0 0)
   )
+  (junction (at 231.14 118.11) (diameter 0) (color 0 0 0 0)
+  )
   (junction (at 64.77 63.5) (diameter 0) (color 0 0 0 0)
   )
@@
   )
   (junction (at 129.54 144.78) (diameter 0) (color 0 0 0 0)
-  )
-  (junction (at 231.14 121.92) (diameter 0) (color 0 0 0 0)
-  )
-  (junction (at 77.47 110.49) (diameter 0) (color 0 0 0 0)
   )
   (junction (at 210.82 99.06) (diameter 0) (color 0 0 0 0)
@@
     (stroke (width 0) (type default))
   )
-  (wire (pts (xy 189.23 113.03) (xy 189.23 121.92))
+  (wire (pts (xy 189.23 113.03) (xy 189.23 118.11))
     (stroke (width 0) (type default))
   )
@@
     (stroke (width 0) (type default))
   )
-  (wire (pts (xy 247.65 74.93) (xy 247.65 121.92))
+  (wire (pts (xy 247.65 74.93) (xy 247.65 118.11))
     (stroke (width 0) (type default))
   )
@@
     (stroke (width 0) (type default))
   )
-  (wire (pts (xy 77.47 110.49) (xy 93.98 110.49))
+  (wire (pts (xy 77.47 118.11) (xy 93.98 118.11))
     (stroke (width 0) (type default))
   )
@@
     (stroke (width 0) (type default))
   )
-  (wire (pts (xy 189.23 121.92) (xy 231.14 121.92))
+  (wire (pts (xy 189.23 118.11) (xy 231.14 118.11))
     (stroke (width 0) (type default))
   )
@@
     (stroke (width 0) (type default))
   )
-  (wire (pts (xy 35.56 110.49) (xy 77.47 110.49))
+  (wire (pts (xy 35.56 118.11) (xy 77.47 118.11))
     (stroke (width 0) (type default))
   )
@@
     (stroke (width 0) (type default))
   )
-  (wire (pts (xy 231.14 113.03) (xy 231.14 121.92))
+  (wire (pts (xy 231.14 113.03) (xy 231.14 118.11))
     (stroke (width 0) (type default))
   )
@@
     (stroke (width 0) (type default))
   )
+  (wire (pts (xy 35.56 118.11) (xy 35.56 110.49))
+    (stroke (width 0) (type default))
+  )
   (wire (pts (xy 25.4 158.75) (xy 25.4 63.5))
+    (stroke (width 0) (type default))
+  )
+  (wire (pts (xy 77.47 118.11) (xy 77.47 110.49))
     (stroke (width 0) (type default))
   )
@@
     (stroke (width 0) (type default))
   )
-  (wire (pts (xy 93.98 107.95) (xy 93.98 110.49))
+  (wire (pts (xy 93.98 107.95) (xy 93.98 118.11))
     (stroke (width 0) (type default))
   )
@@
     (stroke (width 0) (type default))
   )
-  (wire (pts (xy 247.65 121.92) (xy 231.14 121.92))
+  (wire (pts (xy 247.65 118.11) (xy 231.14 118.11))
     (stroke (width 0) (type default))
   )
