File: 8.0/Projects/Master of Dungeons Multilayer/Dimmers.kicad_sch (KiCad schematic)
At the start: 24 parts, among them Q1 IRLML6244, Q14 IRLML6244, Q3 IRLML6244, Q5 IRLML6244

Commit message: update
Parts:
- renumbered C5 to C15, C1 to C16, C3 to C17, D11 to D14, D9 to D15, D5 to D16, D6 to D17, D4 to LED18, D10 to LED19, D1 to LED20, D2 to LED21, Q5 to Q15, Q1 to Q16, Q3 to Q17, R18 to R22, R5 to R23, R1 to R24, R17 to R25, dim3 to dim1, dim4 to dim2, dim1 to dim3, dim2 to dim4

Commit message: up
Parts:
- renumbered C14 to C24, C15 to C25, C16 to C26, C17 to C27, R22 to R26, R23 to R27, R24 to R28, R25 to R29
Changed lines of the file:
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@@
 		(dnp no)
 		(fields_autoplaced yes)
-		(property "Reference" "C15"
+		(property "Reference" "C25"
 			(at 130.81 153.67 90)
 			(effects
@@
 			(project "Master of Dungeons Multilayer"
 				(path "/e447b28f-c2ac-4923-9678-16831d5b7ae9/69c497f5-faba-4d88-8d71-57d6ab81a6aa"
-					(reference "C15")
+					(reference "C25")
 					(unit 1)
 				)
@@
 		(dnp no)
 		(fields_autoplaced yes)
-		(property "Reference" "#PWR089"
+		(property "Reference" "#PWR095"
 			(at 106.68 106.68 0)
 			(effects
@@
 			(project "Master of Dungeons Multilayer"
 				(path "/e447b28f-c2ac-4923-9678-16831d5b7ae9/69c497f5-faba-4d88-8d71-57d6ab81a6aa"
-					(reference "#PWR089")
+					(reference "#PWR095")
 					(unit 1)
 				)
@@
 		(dnp no)
 		(fields_autoplaced yes)
-		(property "Reference" "#PWR097"
+		(property "Reference" "#PWR0103"
 			(at 146.05 130.81 0)
 			(effects
@@
 			(project "Master of Dungeons Multilayer"
 				(path "/e447b28f-c2ac-4923-9678-16831d5b7ae9/69c497f5-faba-4d88-8d71-57d6ab81a6aa"
-					(reference "#PWR097")
+					(reference "#PWR0103")
 					(unit 1)
 				)
@@
 		(dnp no)
 		(fields_autoplaced yes)
-		(property "Reference" "R23"
+		(property "Reference" "R27"
 			(at 130.81 139.7 90)
 			(effects
@@
 			(project "Master of Dungeons Multilayer"
 				(path "/e447b28f-c2ac-4923-9678-16831d5b7ae9/69c497f5-faba-4d88-8d71-57d6ab81a6aa"
-					(reference "R23")
+					(reference "R27")
 					(unit 1)
 				)
@@
 		(dnp no)
 		(fields_autoplaced yes)
-		(property "Reference" "#PWR092"
+		(property "Reference" "#PWR098"
 			(at 107.95 68.58 0)
 			(effects
@@
 			(project "Master of Dungeons Multilayer"
 				(path "/e447b28f-c2ac-4923-9678-16831d5b7ae9/69c497f5-faba-4d88-8d71-57d6ab81a6aa"
-					(reference "#PWR092")
+					(reference "#PWR098")
 					(unit 1)
 				)
@@
 		(dnp no)
 		(fields_autoplaced yes)
-		(property "Reference" "C16"
+		(property "Reference" "C26"
 			(at 132.08 40.64 90)
 			(effects
@@
 			(project "Master of Dungeons Multilayer"
 				(path "/e447b28f-c2ac-4923-9678-16831d5b7ae9/69c497f5-faba-4d88-8d71-57d6ab81a6aa"
-					(reference "C16")
+					(reference "C26")
 					(unit 1)
 				)
@@
 		(dnp no)
 		(fields_autoplaced yes)
-		(property "Reference" "#PWR093"
+		(property "Reference" "#PWR099"
 			(at 127 127 0)
 			(effects
@@
 			(project "Master of Dungeons Multilayer"
 				(path "/e447b28f-c2ac-4923-9678-16831d5b7ae9/69c497f5-faba-4d88-8d71-57d6ab81a6aa"
-					(reference "#PWR093")
+					(reference "#PWR099")
 					(unit 1)
 				)
@@
 		(dnp no)
 		(fields_autoplaced yes)
-		(property "Reference" "#PWR098"
+		(property "Reference" "#PWR0104"
 			(at 146.05 170.18 0)
 			(effects
@@
 			(project "Master of Dungeons Multilayer"
 				(path "/e447b28f-c2ac-4923-9678-16831d5b7ae9/69c497f5-faba-4d88-8d71-57d6ab81a6aa"
-					(reference "#PWR098")
+					(reference "#PWR0104")
 					(unit 1)
 				)
@@
 		(dnp no)
 		(fields_autoplaced yes)
-		(property "Reference" "C14"
+		(property "Reference" "C24"
 			(at 130.81 114.3 90)
 			(effects
@@
 			(project "Master of Dungeons Multilayer"
 				(path "/e447b28f-c2ac-4923-9678-16831d5b7ae9/69c497f5-faba-4d88-8d71-57d6ab81a6aa"
-					(reference "C14")
+					(reference "C24")
 					(unit 1)
 				)
@@
 		(dnp no)
 		(fields_autoplaced yes)
-		(property "Reference" "R24"
+		(property "Reference" "R28"
 			(at 132.08 26.67 90)
 			(effects
@@
 			(project "Master of Dungeons Multilayer"
 				(path "/e447b28f-c2ac-4923-9678-16831d5b7ae9/69c497f5-faba-4d88-8d71-57d6ab81a6aa"
-					(reference "R24")
+					(reference "R28")
 					(unit 1)
 				)
@@
 		(dnp no)
 		(fields_autoplaced yes)
-		(property "Reference" "#PWR094"
+		(property "Reference" "#PWR0100"
 			(at 127 166.37 0)
 			(effects
@@
 			(project "Master of Dungeons Multilayer"
 				(path "/e447b28f-c2ac-4923-9678-16831d5b7ae9/69c497f5-faba-4d88-8d71-57d6ab81a6aa"
-					(reference "#PWR094")
+					(reference "#PWR0100")
 					(unit 1)
 				)
@@
 		(dnp no)
 		(fields_autoplaced yes)
-		(property "Reference" "#PWR0100"
+		(property "Reference" "#PWR0106"
 			(at 147.32 92.71 0)
 			(effects
@@
 			(project "Master of Dungeons Multilayer"
 				(path "/e447b28f-c2ac-4923-9678-16831d5b7ae9/69c497f5-faba-4d88-8d71-57d6ab81a6aa"
-					(reference "#PWR0100")
+					(reference "#PWR0106")
 					(unit 1)
 				)
@@
 		(dnp no)
 		(fields_autoplaced yes)
-		(property "Reference" "#PWR095"
+		(property "Reference" "#PWR0101"
 			(at 128.27 53.34 0)
 			(effects
@@
 			(project "Master of Dungeons Multilayer"
 				(path "/e447b28f-c2ac-4923-9678-16831d5b7ae9/69c497f5-faba-4d88-8d71-57d6ab81a6aa"
-					(reference "#PWR095")
+					(reference "#PWR0101")
 					(unit 1)
 				)
@@
 		(dnp no)
 		(fields_autoplaced yes)
-		(property "Reference" "R25"
+		(property "Reference" "R29"
 			(at 132.08 62.23 90)
 			(effects
@@
 			(project "Master of Dungeons Multilayer"
 				(path "/e447b28f-c2ac-4923-9678-16831d5b7ae9/69c497f5-faba-4d88-8d71-57d6ab81a6aa"
-					(reference "R25")
+					(reference "R29")
 					(unit 1)
 				)
@@
 		(dnp no)
 		(fields_autoplaced yes)
-		(property "Reference" "#PWR090"
+		(property "Reference" "#PWR096"
 			(at 106.68 146.05 0)
 			(effects
@@
 			(project "Master of Dungeons Multilayer"
 				(path "/e447b28f-c2ac-4923-9678-16831d5b7ae9/69c497f5-faba-4d88-8d71-57d6ab81a6aa"
-					(reference "#PWR090")
+					(reference "#PWR096")
 					(unit 1)
 				)
@@
 		(dnp no)
 		(fields_autoplaced yes)
-		(property "Reference" "R22"
+		(property "Reference" "R26"
 			(at 130.81 100.33 90)
 			(effects
@@
 			(project "Master of Dungeons Multilayer"
 				(path "/e447b28f-c2ac-4923-9678-16831d5b7ae9/69c497f5-faba-4d88-8d71-57d6ab81a6aa"
-					(reference "R22")
+					(reference "R26")
 					(unit 1)
 				)
@@
 		(dnp no)
 		(fields_autoplaced yes)
-		(property "Reference" "#PWR099"
+		(property "Reference" "#PWR0105"
 			(at 147.32 57.15 0)
 			(effects
@@
 			(project "Master of Dungeons Multilayer"
 				(path "/e447b28f-c2ac-4923-9678-16831d5b7ae9/69c497f5-faba-4d88-8d71-57d6ab81a6aa"
-					(reference "#PWR099")
+					(reference "#PWR0105")
 					(unit 1)
 				)
@@
 		(dnp no)
 		(fields_autoplaced yes)
-		(property "Reference" "C17"
+		(property "Reference" "C27"
 			(at 132.08 76.2 90)
 			(effects
@@
 			(project "Master of Dungeons Multilayer"
 				(path "/e447b28f-c2ac-4923-9678-16831d5b7ae9/69c497f5-faba-4d88-8d71-57d6ab81a6aa"
-					(reference "C17")
+					(reference "C27")
 					(unit 1)
 				)
@@
 		(dnp no)
 		(fields_autoplaced yes)
-		(property "Reference" "#PWR091"
+		(property "Reference" "#PWR097"
 			(at 107.95 33.02 0)
 			(effects
@@
 			(project "Master of Dungeons Multilayer"
 				(path "/e447b28f-c2ac-4923-9678-16831d5b7ae9/69c497f5-faba-4d88-8d71-57d6ab81a6aa"
-					(reference "#PWR091")
+					(reference "#PWR097")
 					(unit 1)
 				)
@@
 		(dnp no)
 		(fields_autoplaced yes)
-		(property "Reference" "#PWR096"
+		(property "Reference" "#PWR0102"
 			(at 128.27 88.9 0)
 			(effects
@@
 			(project "Master of Dungeons Multilayer"
 				(path "/e447b28f-c2ac-4923-9678-16831d5b7ae9/69c497f5-faba-4d88-8d71-57d6ab81a6aa"
-					(reference "#PWR096")
-					(unit 1)
-				)
+					(reference "#PWR0102")
+					(unit 1)
+				)
