File: 8.0/Projects/Master of Dungeons Multilayer/Sens_Inputs.kicad_sch (KiCad schematic)
At the start: 12 parts

Commit message: update
Parts:
- renumbered R3 to R14, R14 to R15, R15 to R16, R16 to R17
Changed lines of the file:
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@@
 		(dnp no)
 		(fields_autoplaced yes)
-		(property "Reference" "#PWR076"
+		(property "Reference" "#PWR064"
 			(at 115.57 158.75 0)
 			(effects
@@
 			(project "Master of Dungeons Multilayer"
 				(path "/e447b28f-c2ac-4923-9678-16831d5b7ae9/14695e2c-744a-4251-8a70-014f333efa9c"
-					(reference "#PWR076")
+					(reference "#PWR064")
 					(unit 1)
 				)
@@
 		(dnp no)
 		(fields_autoplaced yes)
-		(property "Reference" "#PWR073"
+		(property "Reference" "#PWR063"
 			(at 115.57 124.46 0)
 			(effects
@@
 			(project "Master of Dungeons Multilayer"
 				(path "/e447b28f-c2ac-4923-9678-16831d5b7ae9/14695e2c-744a-4251-8a70-014f333efa9c"
-					(reference "#PWR073")
+					(reference "#PWR063")
 					(unit 1)
 				)
@@
 		(dnp no)
 		(fields_autoplaced yes)
-		(property "Reference" "#PWR075"
+		(property "Reference" "#PWR060"
 			(at 99.06 134.62 0)
 			(effects
@@
 			(project "Master of Dungeons Multilayer"
 				(path "/e447b28f-c2ac-4923-9678-16831d5b7ae9/14695e2c-744a-4251-8a70-014f333efa9c"
-					(reference "#PWR075")
+					(reference "#PWR060")
 					(unit 1)
 				)
@@
 		(dnp no)
 		(fields_autoplaced yes)
-		(property "Reference" "#PWR074"
+		(property "Reference" "#PWR067"
 			(at 115.57 133.35 0)
 			(effects
@@
 			(project "Master of Dungeons Multilayer"
 				(path "/e447b28f-c2ac-4923-9678-16831d5b7ae9/14695e2c-744a-4251-8a70-014f333efa9c"
-					(reference "#PWR074")
+					(reference "#PWR067")
 					(unit 1)
 				)
@@
 		(dnp no)
 		(fields_autoplaced yes)
-		(property "Reference" "#PWR077"
+		(property "Reference" "#PWR068"
 			(at 115.57 167.64 0)
 			(effects
@@
 			(project "Master of Dungeons Multilayer"
 				(path "/e447b28f-c2ac-4923-9678-16831d5b7ae9/14695e2c-744a-4251-8a70-014f333efa9c"
-					(reference "#PWR077")
+					(reference "#PWR068")
 					(unit 1)
 				)
@@
 		(dnp no)
 		(fields_autoplaced yes)
-		(property "Reference" "#PWR013"
+		(property "Reference" "#PWR061"
 			(at 115.57 57.15 0)
 			(effects
@@
 			(project "Master of Dungeons Multilayer"
 				(path "/e447b28f-c2ac-4923-9678-16831d5b7ae9/14695e2c-744a-4251-8a70-014f333efa9c"
-					(reference "#PWR013")
+					(reference "#PWR061")
 					(unit 1)
 				)
@@
 		(dnp no)
 		(fields_autoplaced yes)
-		(property "Reference" "#PWR071"
+		(property "Reference" "#PWR066"
 			(at 115.57 99.06 0)
 			(effects
@@
 			(project "Master of Dungeons Multilayer"
 				(path "/e447b28f-c2ac-4923-9678-16831d5b7ae9/14695e2c-744a-4251-8a70-014f333efa9c"
-					(reference "#PWR071")
+					(reference "#PWR066")
 					(unit 1)
 				)
@@
 		(dnp no)
 		(fields_autoplaced yes)
-		(property "Reference" "#PWR070"
+		(property "Reference" "#PWR062"
 			(at 115.57 90.17 0)
 			(effects
@@
 			(project "Master of Dungeons Multilayer"
 				(path "/e447b28f-c2ac-4923-9678-16831d5b7ae9/14695e2c-744a-4251-8a70-014f333efa9c"
-					(reference "#PWR070")
+					(reference "#PWR062")
 					(unit 1)
 				)
@@
 		(dnp no)
 		(fields_autoplaced yes)
-		(property "Reference" "R15"
+		(property "Reference" "R16"
 			(at 101.6 116.8399 0)
 			(effects
@@
 			(project "Master of Dungeons Multilayer"
 				(path "/e447b28f-c2ac-4923-9678-16831d5b7ae9/14695e2c-744a-4251-8a70-014f333efa9c"
-					(reference "R15")
+					(reference "R16")
 					(unit 1)
 				)
@@
 		(dnp no)
 		(fields_autoplaced yes)
-		(property "Reference" "#PWR041"
+		(property "Reference" "#PWR065"
 			(at 115.57 66.04 0)
 			(effects
@@
 			(project "Master of Dungeons Multilayer"
 				(path "/e447b28f-c2ac-4923-9678-16831d5b7ae9/14695e2c-744a-4251-8a70-014f333efa9c"
-					(reference "#PWR041")
+					(reference "#PWR065")
 					(unit 1)
 				)
@@
 		(dnp no)
 		(fields_autoplaced yes)
-		(property "Reference" "#PWR069"
+		(property "Reference" "#PWR058"
 			(at 99.06 66.04 0)
 			(effects
@@
 			(project "Master of Dungeons Multilayer"
 				(path "/e447b28f-c2ac-4923-9678-16831d5b7ae9/14695e2c-744a-4251-8a70-014f333efa9c"
-					(reference "#PWR069")
+					(reference "#PWR058")
 					(unit 1)
 				)
@@
 		(dnp no)
 		(fields_autoplaced yes)
-		(property "Reference" "R16"
+		(property "Reference" "R17"
 			(at 101.6 151.1299 0)
 			(effects
@@
 			(project "Master of Dungeons Multilayer"
 				(path "/e447b28f-c2ac-4923-9678-16831d5b7ae9/14695e2c-744a-4251-8a70-014f333efa9c"
-					(reference "R16")
+					(reference "R17")
 					(unit 1)
 				)
@@
 		(dnp no)
 		(fields_autoplaced yes)
-		(property "Reference" "R3"
+		(property "Reference" "R14"
 			(at 101.6 49.5299 0)
 			(effects
@@
 			(project "Master of Dungeons Multilayer"
 				(path "/e447b28f-c2ac-4923-9678-16831d5b7ae9/14695e2c-744a-4251-8a70-014f333efa9c"
-					(reference "R3")
+					(reference "R14")
 					(unit 1)
 				)
@@
 		(dnp no)
 		(fields_autoplaced yes)
-		(property "Reference" "#PWR072"
+		(property "Reference" "#PWR059"
 			(at 99.06 100.33 0)
 			(effects
@@
 			(project "Master of Dungeons Multilayer"
 				(path "/e447b28f-c2ac-4923-9678-16831d5b7ae9/14695e2c-744a-4251-8a70-014f333efa9c"
-					(reference "#PWR072")
+					(reference "#PWR059")
 					(unit 1)
 				)
@@
 		(dnp no)
 		(fields_autoplaced yes)
-		(property "Reference" "R14"
+		(property "Reference" "R15"
 			(at 101.6 82.5499 0)
 			(effects
@@
 			(project "Master of Dungeons Multilayer"
 				(path "/e447b28f-c2ac-4923-9678-16831d5b7ae9/14695e2c-744a-4251-8a70-014f333efa9c"
-					(reference "R14")
+					(reference "R15")
 					(unit 1)
 				)
@@
 		(dnp no)
 		(fields_autoplaced yes)
-		(property "Reference" "#PWR040"
+		(property "Reference" "#PWR057"
 			(at 99.06 33.02 0)
 			(effects
@@
 			(project "Master of Dungeons Multilayer"
 				(path "/e447b28f-c2ac-4923-9678-16831d5b7ae9/14695e2c-744a-4251-8a70-014f333efa9c"
-					(reference "#PWR040")
-					(unit 1)
-				)
+					(reference "#PWR057")
+					(unit 1)
+				)

Commit message: up
Parts:
- renumbered R14 to R18, R15 to R19, R16 to R20, R17 to R21
Changed lines of the file:
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@@
 		(dnp no)
 		(fields_autoplaced yes)
-		(property "Reference" "#PWR064"
+		(property "Reference" "#PWR070"
 			(at 115.57 158.75 0)
 			(effects
@@
 			(project "Master of Dungeons Multilayer"
 				(path "/e447b28f-c2ac-4923-9678-16831d5b7ae9/14695e2c-744a-4251-8a70-014f333efa9c"
-					(reference "#PWR064")
+					(reference "#PWR070")
 					(unit 1)
 				)
@@
 		(dnp no)
 		(fields_autoplaced yes)
-		(property "Reference" "#PWR063"
+		(property "Reference" "#PWR069"
 			(at 115.57 124.46 0)
 			(effects
@@
 			(project "Master of Dungeons Multilayer"
 				(path "/e447b28f-c2ac-4923-9678-16831d5b7ae9/14695e2c-744a-4251-8a70-014f333efa9c"
-					(reference "#PWR063")
+					(reference "#PWR069")
 					(unit 1)
 				)
@@
 		(dnp no)
 		(fields_autoplaced yes)
-		(property "Reference" "#PWR060"
+		(property "Reference" "#PWR066"
 			(at 99.06 134.62 0)
 			(effects
@@
 			(project "Master of Dungeons Multilayer"
 				(path "/e447b28f-c2ac-4923-9678-16831d5b7ae9/14695e2c-744a-4251-8a70-014f333efa9c"
-					(reference "#PWR060")
+					(reference "#PWR066")
 					(unit 1)
 				)
@@
 		(dnp no)
 		(fields_autoplaced yes)
-		(property "Reference" "#PWR067"
+		(property "Reference" "#PWR073"
 			(at 115.57 133.35 0)
 			(effects
@@
 			(project "Master of Dungeons Multilayer"
 				(path "/e447b28f-c2ac-4923-9678-16831d5b7ae9/14695e2c-744a-4251-8a70-014f333efa9c"
-					(reference "#PWR067")
+					(reference "#PWR073")
 					(unit 1)
 				)
@@
 		(dnp no)
 		(fields_autoplaced yes)
-		(property "Reference" "#PWR068"
+		(property "Reference" "#PWR074"
 			(at 115.57 167.64 0)
 			(effects
@@
 			(project "Master of Dungeons Multilayer"
 				(path "/e447b28f-c2ac-4923-9678-16831d5b7ae9/14695e2c-744a-4251-8a70-014f333efa9c"
-					(reference "#PWR068")
+					(reference "#PWR074")
 					(unit 1)
 				)
@@
 		(dnp no)
 		(fields_autoplaced yes)
-		(property "Reference" "#PWR061"
+		(property "Reference" "#PWR067"
 			(at 115.57 57.15 0)
 			(effects
@@
 			(project "Master of Dungeons Multilayer"
 				(path "/e447b28f-c2ac-4923-9678-16831d5b7ae9/14695e2c-744a-4251-8a70-014f333efa9c"
-					(reference "#PWR061")
+					(reference "#PWR067")
 					(unit 1)
 				)
@@
 		(dnp no)
 		(fields_autoplaced yes)
-		(property "Reference" "#PWR066"
+		(property "Reference" "#PWR072"
 			(at 115.57 99.06 0)
 			(effects
@@
 			(project "Master of Dungeons Multilayer"
 				(path "/e447b28f-c2ac-4923-9678-16831d5b7ae9/14695e2c-744a-4251-8a70-014f333efa9c"
-					(reference "#PWR066")
+					(reference "#PWR072")
 					(unit 1)
 				)
@@
 		(dnp no)
 		(fields_autoplaced yes)
-		(property "Reference" "#PWR062"
+		(property "Reference" "#PWR068"
 			(at 115.57 90.17 0)
 			(effects
@@
 			(project "Master of Dungeons Multilayer"
 				(path "/e447b28f-c2ac-4923-9678-16831d5b7ae9/14695e2c-744a-4251-8a70-014f333efa9c"
-					(reference "#PWR062")
+					(reference "#PWR068")
 					(unit 1)
 				)
@@
 		(dnp no)
 		(fields_autoplaced yes)
-		(property "Reference" "R16"
+		(property "Reference" "R20"
 			(at 101.6 116.8399 0)
 			(effects
@@
 			(project "Master of Dungeons Multilayer"
 				(path "/e447b28f-c2ac-4923-9678-16831d5b7ae9/14695e2c-744a-4251-8a70-014f333efa9c"
-					(reference "R16")
+					(reference "R20")
 					(unit 1)
 				)
@@
 		(dnp no)
 		(fields_autoplaced yes)
-		(property "Reference" "#PWR065"
+		(property "Reference" "#PWR071"
 			(at 115.57 66.04 0)
 			(effects
@@
 			(project "Master of Dungeons Multilayer"
 				(path "/e447b28f-c2ac-4923-9678-16831d5b7ae9/14695e2c-744a-4251-8a70-014f333efa9c"
-					(reference "#PWR065")
+					(reference "#PWR071")
 					(unit 1)
 				)
@@
 		(dnp no)
 		(fields_autoplaced yes)
-		(property "Reference" "#PWR058"
+		(property "Reference" "#PWR064"
 			(at 99.06 66.04 0)
 			(effects
@@
 			(project "Master of Dungeons Multilayer"
 				(path "/e447b28f-c2ac-4923-9678-16831d5b7ae9/14695e2c-744a-4251-8a70-014f333efa9c"
-					(reference "#PWR058")
+					(reference "#PWR064")
 					(unit 1)
 				)
@@
 		(dnp no)
 		(fields_autoplaced yes)
-		(property "Reference" "R17"
+		(property "Reference" "R21"
 			(at 101.6 151.1299 0)
 			(effects
@@
 			(project "Master of Dungeons Multilayer"
 				(path "/e447b28f-c2ac-4923-9678-16831d5b7ae9/14695e2c-744a-4251-8a70-014f333efa9c"
-					(reference "R17")
+					(reference "R21")
 					(unit 1)
 				)
@@
 		(dnp no)
 		(fields_autoplaced yes)
-		(property "Reference" "R14"
+		(property "Reference" "R18"
 			(at 101.6 49.5299 0)
 			(effects
@@
 			(project "Master of Dungeons Multilayer"
 				(path "/e447b28f-c2ac-4923-9678-16831d5b7ae9/14695e2c-744a-4251-8a70-014f333efa9c"
-					(reference "R14")
+					(reference "R18")
 					(unit 1)
 				)
@@
 		(dnp no)
 		(fields_autoplaced yes)
-		(property "Reference" "#PWR059"
+		(property "Reference" "#PWR065"
 			(at 99.06 100.33 0)
 			(effects
@@
 			(project "Master of Dungeons Multilayer"
 				(path "/e447b28f-c2ac-4923-9678-16831d5b7ae9/14695e2c-744a-4251-8a70-014f333efa9c"
-					(reference "#PWR059")
+					(reference "#PWR065")
 					(unit 1)
 				)
@@
 		(dnp no)
 		(fields_autoplaced yes)
-		(property "Reference" "R15"
+		(property "Reference" "R19"
 			(at 101.6 82.5499 0)
 			(effects
@@
 			(project "Master of Dungeons Multilayer"
 				(path "/e447b28f-c2ac-4923-9678-16831d5b7ae9/14695e2c-744a-4251-8a70-014f333efa9c"
-					(reference "R15")
+					(reference "R19")
 					(unit 1)
 				)
@@
 		(dnp no)
 		(fields_autoplaced yes)
-		(property "Reference" "#PWR057"
+		(property "Reference" "#PWR063"
 			(at 99.06 33.02 0)
 			(effects
@@
 			(project "Master of Dungeons Multilayer"
 				(path "/e447b28f-c2ac-4923-9678-16831d5b7ae9/14695e2c-744a-4251-8a70-014f333efa9c"
-					(reference "#PWR057")
-					(unit 1)
-				)
+					(reference "#PWR063")
+					(unit 1)
+				)
