File: 8.0/Projects/Master of Dungeons Multilayer/Sens_Outputs.kicad_sch (KiCad schematic)
At the start: 24 parts, among them Q15 IRLML6244, Q16 IRLML6244, Q17 IRLML6244, Q4 IRLML6244

Commit message: update
Parts:
- renumbered C4 to C10, C15 to C11, C16 to C12, C17 to C13, D7 to D10, D15 to D11, D19 to D12, D23 to D13, D8 to LED14, D13 to LED15, D17 to LED16, D21 to LED17, Q4 to Q10, Q15 to Q11, Q16 to Q12, Q17 to Q13, R4 to R18

Commit message: up
Parts:
- renumbered C10 to C20, C11 to C21, C12 to C22, C13 to C23, R18 to R22, R19 to R23, R20 to R24, R21 to R25
