File: 8.0/Projects/Master of Dungeons Multilayer/Master of Dungeons Multilayer.kicad_sch (KiCad schematic)
At the start: 14 parts, among them J1 AudioPlug3, U1 ESP32-WROOM-32E, U2 TPS63060, U3 AP2127K-3.3, U4 TSOP45xx

Commit message: update
Parts:
- R1: renamed from R25; footprint (none) -> Resistor_SMD:R_0805_2012Metric_Pad1.20x1.40mm_HandSolder
- R2: renamed from R24; footprint (none) -> Resistor_SMD:R_0805_2012Metric_Pad1.20x1.40mm_HandSolder
- R3: renamed from R22; footprint (none) -> Resistor_SMD:R_0805_2012Metric_Pad1.20x1.40mm_HandSolder
- R4: renamed from R23; footprint (none) -> Resistor_SMD:R_0805_2012Metric_Pad1.20x1.40mm_HandSolder
- renumbered U2 to U1, U3 to U2, U1 to U3
Changed lines of the file:
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@@
 		(dnp no)
 		(fields_autoplaced yes)
-		(property "Reference" "R24"
+		(property "Reference" "R2"
 			(at 46.99 64.7699 0)
 			(effects
@@
 			)
 		)
-		(property "Footprint" ""
+		(property "Footprint" "Resistor_SMD:R_0805_2012Metric_Pad1.20x1.40mm_HandSolder"
 			(at 42.672 66.04 90)
 			(effects
@@
 			(project "Master of Dungeons Multilayer"
 				(path "/e447b28f-c2ac-4923-9678-16831d5b7ae9"
-					(reference "R24")
+					(reference "R2")
 					(unit 1)
 				)
@@
 		(dnp no)
 		(fields_autoplaced yes)
-		(property "Reference" "U2"
+		(property "Reference" "U1"
 			(at 62.23 154.94 0)
 			(effects
@@
 			(project ""
 				(path "/e447b28f-c2ac-4923-9678-16831d5b7ae9"
-					(reference "U2")
+					(reference "U1")
 					(unit 1)
 				)
@@
 		(on_board yes)
 		(dnp no)
-		(property "Reference" "#PWR099"
+		(property "Reference" "#PWR03"
 			(at 40.64 72.39 0)
 			(effects
@@
 			(project "Master of Dungeons Multilayer"
 				(path "/e447b28f-c2ac-4923-9678-16831d5b7ae9"
-					(reference "#PWR099")
+					(reference "#PWR03")
 					(unit 1)
 				)
@@
 		(dnp no)
 		(fields_autoplaced yes)
-		(property "Reference" "#PWR042"
+		(property "Reference" "#PWR012"
 			(at 133.35 147.32 0)
 			(effects
@@
 			(project "Master of Dungeons Multilayer"
 				(path "/e447b28f-c2ac-4923-9678-16831d5b7ae9"
-					(reference "#PWR042")
+					(reference "#PWR012")
 					(unit 1)
 				)
@@
 		(dnp no)
 		(fields_autoplaced yes)
-		(property "Reference" "#PWR07"
+		(property "Reference" "#PWR016"
 			(at 251.46 45.72 0)
 			(effects
@@
 			(project "Master of Dungeons Multilayer"
 				(path "/e447b28f-c2ac-4923-9678-16831d5b7ae9"
-					(reference "#PWR07")
+					(reference "#PWR016")
 					(unit 1)
 				)
@@
 		(on_board yes)
 		(dnp no)
-		(property "Reference" "#PWR023"
+		(property "Reference" "#PWR09"
 			(at 95.25 63.5 0)
 			(effects
@@
 			(project "Master of Dungeons Multilayer"
 				(path "/e447b28f-c2ac-4923-9678-16831d5b7ae9"
-					(reference "#PWR023")
+					(reference "#PWR09")
 					(unit 1)
 				)
@@
 		(dnp no)
 		(fields_autoplaced yes)
-		(property "Reference" "#PWR05"
+		(property "Reference" "#PWR02"
 			(at 30.48 172.72 0)
 			(effects
@@
 			(project "Master of Dungeons Multilayer"
 				(path "/e447b28f-c2ac-4923-9678-16831d5b7ae9"
-					(reference "#PWR05")
+					(reference "#PWR02")
 					(unit 1)
 				)
@@
 		(dnp no)
 		(fields_autoplaced yes)
-		(property "Reference" "#PWR012"
+		(property "Reference" "#PWR015"
 			(at 251.46 27.94 0)
 			(effects
@@
 			(project "Master of Dungeons Multilayer"
 				(path "/e447b28f-c2ac-4923-9678-16831d5b7ae9"
-					(reference "#PWR012")
+					(reference "#PWR015")
 					(unit 1)
 				)
@@
 		(dnp no)
 		(fields_autoplaced yes)
-		(property "Reference" "#PWR024"
+		(property "Reference" "#PWR08"
 			(at 80.01 166.37 0)
 			(effects
@@
 			(project "Master of Dungeons Multilayer"
 				(path "/e447b28f-c2ac-4923-9678-16831d5b7ae9"
-					(reference "#PWR024")
+					(reference "#PWR08")
 					(unit 1)
 				)
@@
 		(dnp no)
 		(fields_autoplaced yes)
-		(property "Reference" "#PWR0100"
+		(property "Reference" "#PWR01"
 			(at 30.48 49.53 0)
 			(effects
@@
 			(project "Master of Dungeons Multilayer"
 				(path "/e447b28f-c2ac-4923-9678-16831d5b7ae9"
-					(reference "#PWR0100")
+					(reference "#PWR01")
 					(unit 1)
 				)
@@
 		(dnp no)
 		(fields_autoplaced yes)
-		(property "Reference" "#PWR098"
+		(property "Reference" "#PWR010"
 			(at 102.87 45.72 0)
 			(effects
@@
 			(project "Master of Dungeons Multilayer"
 				(path "/e447b28f-c2ac-4923-9678-16831d5b7ae9"
-					(reference "#PWR098")
+					(reference "#PWR010")
 					(unit 1)
 				)
@@
 		(dnp no)
 		(fields_autoplaced yes)
-		(property "Reference" "#PWR027"
+		(property "Reference" "#PWR013"
 			(at 172.72 123.19 0)
 			(effects
@@
 			(project "Master of Dungeons Multilayer"
 				(path "/e447b28f-c2ac-4923-9678-16831d5b7ae9"
-					(reference "#PWR027")
+					(reference "#PWR013")
 					(unit 1)
 				)
@@
 		(dnp no)
 		(fields_autoplaced yes)
-		(property "Reference" "#PWR022"
+		(property "Reference" "#PWR05"
 			(at 60.96 62.23 0)
 			(effects
@@
 			(project "Master of Dungeons Multilayer"
 				(path "/e447b28f-c2ac-4923-9678-16831d5b7ae9"
-					(reference "#PWR022")
+					(reference "#PWR05")
 					(unit 1)
 				)
@@
 		(dnp no)
 		(fields_autoplaced yes)
-		(property "Reference" "#PWR043"
+		(property "Reference" "#PWR011"
 			(at 143.51 143.51 0)
 			(effects
@@
 			(project "Master of Dungeons Multilayer"
 				(path "/e447b28f-c2ac-4923-9678-16831d5b7ae9"
-					(reference "#PWR043")
+					(reference "#PWR011")
 					(unit 1)
 				)
@@
 		(dnp no)
 		(fields_autoplaced yes)
-		(property "Reference" "#PWR06"
+		(property "Reference" "#PWR04"
 			(at 59.69 194.31 0)
 			(effects
@@
 			(project "Master of Dungeons Multilayer"
 				(path "/e447b28f-c2ac-4923-9678-16831d5b7ae9"
-					(reference "#PWR06")
+					(reference "#PWR04")
 					(unit 1)
 				)
@@
 		(dnp no)
 		(fields_autoplaced yes)
-		(property "Reference" "U3"
+		(property "Reference" "U2"
 			(at 74.93 52.0699 90)
 			(effects
@@
 			(project ""
 				(path "/e447b28f-c2ac-4923-9678-16831d5b7ae9"
-					(reference "U3")
+					(reference "U2")
 					(unit 1)
 				)
@@
 		(dnp no)
 		(fields_autoplaced yes)
-		(property "Reference" "R23"
+		(property "Reference" "R4"
 			(at 105.41 71.1199 0)
 			(effects
@@
 			)
 		)
-		(property "Footprint" ""
+		(property "Footprint" "Resistor_SMD:R_0805_2012Metric_Pad1.20x1.40mm_HandSolder"
 			(at 101.092 72.39 90)
 			(effects
@@
 			(project "Master of Dungeons Multilayer"
 				(path "/e447b28f-c2ac-4923-9678-16831d5b7ae9"
-					(reference "R23")
+					(reference "R4")
 					(unit 1)
 				)
@@
 		(dnp no)
 		(fields_autoplaced yes)
-		(property "Reference" "#PWR08"
+		(property "Reference" "#PWR014"
 			(at 176.53 74.93 0)
 			(effects
@@
 			(project "Master of Dungeons Multilayer"
 				(path "/e447b28f-c2ac-4923-9678-16831d5b7ae9"
-					(reference "#PWR08")
+					(reference "#PWR014")
 					(unit 1)
 				)
@@
 		(dnp no)
 		(fields_autoplaced yes)
-		(property "Reference" "U1"
+		(property "Reference" "U3"
 			(at 73.3141 68.58 0)
 			(effects
@@
 			(project ""
 				(path "/e447b28f-c2ac-4923-9678-16831d5b7ae9"
-					(reference "U1")
+					(reference "U3")
 					(unit 1)
 				)
@@
 		(dnp no)
 		(fields_autoplaced yes)
-		(property "Reference" "#PWR025"
+		(property "Reference" "#PWR07"
 			(at 76.2 41.91 0)
 			(effects
@@
 			(project "Master of Dungeons Multilayer"
 				(path "/e447b28f-c2ac-4923-9678-16831d5b7ae9"
-					(reference "#PWR025")
+					(reference "#PWR07")
 					(unit 1)
 				)
@@
 		(dnp no)
 		(fields_autoplaced yes)
-		(property "Reference" "R25"
+		(property "Reference" "R1"
 			(at 38.1 34.29 90)
 			(effects
@@
 			)
 		)
-		(property "Footprint" ""
+		(property "Footprint" "Resistor_SMD:R_0805_2012Metric_Pad1.20x1.40mm_HandSolder"
 			(at 38.1 38.862 90)
 			(effects
@@
 			(project "Master of Dungeons Multilayer"
 				(path "/e447b28f-c2ac-4923-9678-16831d5b7ae9"
-					(reference "R25")
+					(reference "R1")
 					(unit 1)
 				)
@@
 		(dnp no)
 		(fields_autoplaced yes)
-		(property "Reference" "#PWR01"
+		(property "Reference" "#PWR06"
 			(at 71.12 148.59 0)
 			(effects
@@
 			(project ""
 				(path "/e447b28f-c2ac-4923-9678-16831d5b7ae9"
-					(reference "#PWR01")
+					(reference "#PWR06")
 					(unit 1)
 				)
@@
 		(dnp no)
 		(fields_autoplaced yes)
-		(property "Reference" "R22"
+		(property "Reference" "R3"
 			(at 97.79 71.1199 0)
 			(effects
@@
 			)
 		)
-		(property "Footprint" ""
+		(property "Footprint" "Resistor_SMD:R_0805_2012Metric_Pad1.20x1.40mm_HandSolder"
 			(at 93.472 72.39 90)
 			(effects
@@
 			(project ""
 				(path "/e447b28f-c2ac-4923-9678-16831d5b7ae9"
-					(reference "R22")
-					(unit 1)
-				)
+					(reference "R3")
+					(unit 1)
+				)

Commit message: up
Parts:
- added C1, C2: 10uF, Capacitor_SMD:C_0805_2012Metric_Pad1.18x1.45mm_HandSolder, symbol Device:C
- added C10: 100nF, Capacitor_SMD:C_0805_2012Metric_Pad1.18x1.45mm_HandSolder, symbol Device:C
- added C3, C5: 1uF, Capacitor_SMD:C_0805_2012Metric_Pad1.18x1.45mm_HandSolder, symbol Device:C
- added C4: .1uF, Capacitor_SMD:C_0805_2012Metric_Pad1.18x1.45mm_HandSolder, symbol Device:C
- added C6: 10pF, Capacitor_SMD:C_0805_2012Metric_Pad1.18x1.45mm_HandSolder, symbol Device:C
- added C7, C8, C9: 22uF, Capacitor_SMD:C_0805_2012Metric_Pad1.18x1.45mm_HandSolder, symbol Device:C
- added L1: L, Inductor_SMD:L_Coilcraft_XAL4020-XXX, symbol Device:L
- added R3, R6: 1M, Resistor_SMD:R_0805_2012Metric_Pad1.20x1.40mm_HandSolder, symbol Device:R
- added R30: 12K, Resistor_SMD:R_0805_2012Metric_Pad1.20x1.40mm_HandSolder, symbol Device:R
- added R4: 111K, Resistor_SMD:R_0805_2012Metric_Pad1.20x1.40mm_HandSolder, symbol Device:R
- added R8: 470R, Resistor_SMD:R_0805_2012Metric_Pad1.20x1.40mm_HandSolder, symbol Device:R
- PWR1: footprint Connector_JST:JST_XH_S2B-XH-A_1x02_P2.50mm_Horizontal -> Connector_PinHeader_2.54mm:PinHeader_1x02_P2.54mm_Vertical
- renumbered R3 to R5, R4 to R7
Connections:
- net +3.3V: now also C3.1
- net +5V: now also C5.1, C7.1, C8.1, C9.1, R3.2, R6.2, R8.2; no longer U4.3 (Vs)
- net GND: now also U1.11 (PGND), U1.4 (PS/SYNC), C1.1, C10.1, C2.2, C3.2, C4.2, C5.2, C6.2, C7.2, C8.2, C9.2, R30.1, R4.1
- net at U1.1 (L1): now also L1.2
- net at U1.10 (L2): now also L1.1
- net at PWR1.1 (Pin_1), U1.2 (VIN): now also U1.3 (EN), C1.2, C2.1
- net at U1.5 (PG): now also R6.1
- net at U1.6 (VAUX): now also C4.1
- net at U1.8 (FB): now also C6.1, R3.1, R4.2
- net at U2.3 (EN): now also R30.2
- new net: C10.2, R8.1, U4.3 (Vs)
Other:
- moved on the sheet: PWR1, U2

Commit message: Up
Parts:
- removed C1, C2: 10uF, Capacitor_SMD:C_0805_2012Metric_Pad1.18x1.45mm_HandSolder, symbol Device:C
- removed C3, C5: 1uF, Capacitor_SMD:C_0805_2012Metric_Pad1.18x1.45mm_HandSolder, symbol Device:C
- removed C4: .1uF, Capacitor_SMD:C_0805_2012Metric_Pad1.18x1.45mm_HandSolder, symbol Device:C
- removed C6: 10pF, Capacitor_SMD:C_0805_2012Metric_Pad1.18x1.45mm_HandSolder, symbol Device:C
- removed C7, C8, C9: 22uF, Capacitor_SMD:C_0805_2012Metric_Pad1.18x1.45mm_HandSolder, symbol Device:C
- removed L1: L, Inductor_SMD:L_Coilcraft_XAL4020-XXX, symbol Device:L
- removed PWR1: Conn_01x02_Pin, Connector_PinHeader_2.54mm:PinHeader_1x02_P2.54mm_Vertical, symbol Connector:Conn_01x02_Pin
- removed R3, R6: 1M, Resistor_SMD:R_0805_2012Metric_Pad1.20x1.40mm_HandSolder, symbol Device:R
- removed R30: 12K, Resistor_SMD:R_0805_2012Metric_Pad1.20x1.40mm_HandSolder, symbol Device:R
- removed R4: 111K, Resistor_SMD:R_0805_2012Metric_Pad1.20x1.40mm_HandSolder, symbol Device:R
- removed U1: TPS63060, Package_SON:Texas_S-PWSON-N10_ThermalVias, symbol Regulator_Switching:TPS63060
- removed U2: AP2127K-3.3, Package_TO_SOT_SMD:SOT-23-5, symbol Regulator_Linear:AP2127K-3.3
Other:
- added sheet Power (Power.kicad_sch)
