File: 8.0/Projects/Master of Dungeons Multilayer/Master of Dungeons Multilayer.kicad_pcb (KiCad board)
At the start: 4 copper layers, 100 x 100 mm, 124 parts, among them J1 AudioPlug3, Q1 IRLML6244, Q10 IRLML6244, Q11 IRLML6244, Q12 IRLML6244, Q13 IRLML6244, Q14 IRLML6244, Q15 IRLML6244, Q16 IRLML6244, Q17 IRLML6244, Q2 IRLML6244, Q3 IRLML6244, Q4 IRLML6244, Q5 IRLML6244, Q6 IRLML6244, Q7 IRLML6244, Q8 IRLML6244, Q9 IRLML6244, U1 ESP32-WROOM-32E, U2 TPS63060, U3 AP2127K-3.3, U4 TSOP45xx

Commit message: ghj
Routing:
- added copper zone on In2.Cu, net +3.3V
- added copper zone on In1.Cu, net +5V
- added copper zone on F.Cu, net GND
Changed lines of the file:
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@@
 		(net 92)
 	)
+	(zone
+		(net 89)
+		(net_name "GND")
+		(layer "F.Cu")
+		(hatch edge 0.5)
+		(connect_pads
+			(clearance 0.5)
+		)
+		(min_thickness 0.25)
+		(filled_areas_thickness no)
+		(fill
+			(thermal_gap 0.5)
+			(thermal_bridge_width 0.5)
+		)
+		(polygon
+			(pts
+				(xy 100.4 50.3) (xy 199.89 50.3) (xy 199.9 149.89) (xy 100.4 149.84)
+			)
+		)
+	)
+	(zone
+		(net 5)
+		(net_name "+5V")
+		(layer "In1.Cu")
+		(hatch edge 0.5)
+		(priority 1)
+		(connect_pads
+			(clearance 0.5)
+		)
+		(min_thickness 0.25)
+		(filled_areas_thickness no)
+		(fill
+			(thermal_gap 0.5)
+			(thermal_bridge_width 0.5)
+		)
+		(polygon
+			(pts
+				(xy 100.4 50.3) (xy 199.89 50.3) (xy 199.9 149.89) (xy 100.4 149.84)
+			)
+		)
+	)
+	(zone
+		(net 67)
+		(net_name "+3.3V")
+		(layer "In2.Cu")
+		(hatch edge 0.5)
+		(priority 2)
+		(connect_pads
+			(clearance 0.5)
+		)
+		(min_thickness 0.25)
+		(filled_areas_thickness no)
+		(fill
+			(thermal_gap 0.5)
+			(thermal_bridge_width 0.5)
+		)
+		(polygon
+			(pts
+				(xy 100.4 50.31) (xy 199.89 50.3) (xy 199.9 149.89) (xy 100.4 149.84)
+			)
+		)
+	)
 )

Commit message: update
Parts:
- added R1: 470R, Resistor_SMD:R_0805_2012Metric_Pad1.20x1.40mm_HandSolder, F.Cu at (72.1, 39.5)
- added R2: 12K, Resistor_SMD:R_0805_2012Metric_Pad1.20x1.40mm_HandSolder, F.Cu at (72.1, 50.2)
- added R3: 12K, Resistor_SMD:R_0805_2012Metric_Pad1.20x1.40mm_HandSolder, F.Cu at (63.8, 44.5)
- added R4: 470R, Resistor_SMD:R_0805_2012Metric_Pad1.20x1.40mm_HandSolder, F.Cu at (63.6, 39.5)
- moved TxRxGND1 130.9 mm to (48.7, 42.0), turned to 0 degrees
- moved J1 114.7 mm to (70.2, 167.8)
- moved BOOT1 106.6 mm to (59.5, 44.9)
- moved U1 67.6 mm to (121.8, 43.3)
- moved U2 66.5 mm to (121.7, 49.1)
- moved RST1 65.9 mm to (68.0, 44.9), turned to -90 degrees
- moved U4 65.6 mm to (55.0, 170.0)
- moved sensOut4 60.2 mm to (46.6, 138.0)
- moved sensOut3 60.2 mm to (46.6, 127.1)
- moved sensOut2 60.1 mm to (46.6, 116.1)
- moved sensOut1 60.1 mm to (46.6, 105.2)
- moved sens2 60.0 mm to (46.5, 66.0)
- moved sens1 60.0 mm to (46.5, 55.0)
- moved sens4 60.0 mm to (46.5, 87.9)
- moved sens3 60.0 mm to (46.5, 76.9)
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- renumbered C6 to C1, C4 to C10, C15 to C11, C16 to C12, C17 to C13, C5 to C15, C1 to C16, C3 to C17, C7 to C2, C8 to C3, C9 to C4, C10 to C5, C11 to C6, C2 to C7, C12 to C8, C13 to C9, D3 to D1, D7 to D10, D15 to D11, D19 to D12, D23 to D13, D11 to D14, D9 to D15, D5 to D16, D6 to D17, D12 to D2, D14 to D3, D16 to D4, D18 to D5, D20 to D6, D22 to D7, D24 to D8, D26 to D9, D8 to LED14, D13 to LED15, D17 to LED16, D21 to LED17, D4 to LED18, D10 to LED19, D1 to LED20, D2 to LED21, Q2 to Q1, Q4 to Q10, Q15 to Q11, Q16 to Q12, Q17 to Q13, Q5 to Q15, Q1 to Q16, Q3 to Q17, Q6 to Q2, Q7 to Q3, Q8 to Q4, Q9 to Q5, Q10 to Q6, Q11 to Q7, Q12 to Q8, Q13 to Q9, R3 to R14, R14 to R15, R15 to R16, R16 to R17, R4 to R18, R18 to R22, R5 to R23, R1 to R24, R17 to R25, R2 to R5, U2 to U1, U3 to U2, U1 to U3, dim3 to dim1, dim4 to dim2, dim1 to dim3, dim2 to dim4
Connections:
- I2C1 pad 1: +5V -> GND
- I2C1 pad 2: GND -> +5V
Routing:
- net +5V: track 85.6 -> 0.00 mm, vias 19 -> 0
- net port1: track 81.4 -> 0.00 mm
- net sensOut4: track 79.7 -> 0.00 mm
- net port2: track 74.6 -> 0.00 mm
- net dim2: track 72.3 -> 0.00 mm
- net dim1: track 71.7 -> 0.00 mm
- net dim4: track 71.5 -> 0.00 mm
- net sensOut3: track 71.4 -> 0.00 mm
- net dim3: track 69.4 -> 0.00 mm
- net port3: track 68.2 -> 0.00 mm
- net sensOut2: track 64.8 -> 0.00 mm
- net port4: track 62.0 -> 0.00 mm
- net port5: track 55.3 -> 0.00 mm
- net sensOut1: track 50.6 -> 0.00 mm
- net sens4: track 49.3 -> 0.00 mm
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- removed copper zone on In2.Cu, net +3.3V
- removed copper zone on In1.Cu, net +5V
- removed copper zone on F.Cu, net GND
Other:
- board size 100 x 100 mm -> 110 x 145 mm

Commit message: up
Parts:
- added C1: 10uF, Capacitor_SMD:C_0805_2012Metric_Pad1.18x1.45mm_HandSolder, B.Cu at (127.6, 46.5)
- added C10: 100nF, Capacitor_SMD:C_0805_2012Metric_Pad1.18x1.45mm_HandSolder, F.Cu at (54.9, 170.3)
- added C2: 10uF, Capacitor_SMD:C_0805_2012Metric_Pad1.18x1.45mm_HandSolder, B.Cu at (127.6, 44.5)
- added C3: 1uF, Capacitor_SMD:C_0805_2012Metric_Pad1.18x1.45mm_HandSolder, B.Cu at (106.2, 51.7)
- added C4: .1uF, Capacitor_SMD:C_0805_2012Metric_Pad1.18x1.45mm_HandSolder, B.Cu at (120.3, 50.0)
- added C5: 1uF, Capacitor_SMD:C_0805_2012Metric_Pad1.18x1.45mm_HandSolder, B.Cu at (110.4, 49.9)
- added C6: 10pF, Capacitor_SMD:C_0805_2012Metric_Pad1.18x1.45mm_HandSolder, B.Cu at (115.8, 49.9)
- added C7: 22uF, Capacitor_SMD:C_0805_2012Metric_Pad1.18x1.45mm_HandSolder, B.Cu at (112.9, 44.1)
- added C8: 22uF, Capacitor_SMD:C_0805_2012Metric_Pad1.18x1.45mm_HandSolder, B.Cu at (109.9, 44.1)
- added C9: 22uF, Capacitor_SMD:C_0805_2012Metric_Pad1.18x1.45mm_HandSolder, B.Cu at (106.9, 44.1)
- added L1: L, Inductor_SMD:L_Coilcraft_XAL4020-XXX, B.Cu at (122.7, 40.4)
- added R3: 1M, Resistor_SMD:R_0805_2012Metric_Pad1.20x1.40mm_HandSolder, B.Cu at (116.6, 45.6)
- added R30: 12K, Resistor_SMD:R_0805_2012Metric_Pad1.20x1.40mm_HandSolder, B.Cu at (110.4, 57.9)
- added R4: 111K, Resistor_SMD:R_0805_2012Metric_Pad1.20x1.40mm_HandSolder, B.Cu at (118.0, 49.9)
- added R6: 1M, Resistor_SMD:R_0805_2012Metric_Pad1.20x1.40mm_HandSolder, B.Cu at (124.4, 50.0)
- added R8: 470R, Resistor_SMD:R_0805_2012Metric_Pad1.20x1.40mm_HandSolder, F.Cu at (55.0, 167.3)
- PWR1: footprint Connector_JST:JST_XH_S2B-XH-A_1x02_P2.50mm_Horizontal -> Connector_PinHeader_2.54mm:PinHeader_1x02_P2.54mm_Vertical
- moved PWR1 22.7 mm to (119.4, 56.1)
- moved U2 13.3 mm to (109.3, 53.9)
- moved LED5 5.89 mm to (126.1, 108.0)
- moved R16 5.89 mm to (124.3, 75.6)
- moved Q9 5.89 mm to (131.8, 64.6)
- moved R17 5.89 mm to (124.4, 64.7)
- moved C12 5.89 mm to (131.3, 120.9)
- moved C13 5.89 mm to (131.2, 113.2)
- moved C14 5.89 mm to (131.4, 104.5)
- moved C16 5.89 mm to (133.4, 82.2)
- moved C18 5.89 mm to (133.5, 71.0)
- moved C19 5.89 mm to (133.5, 59.9)
- moved C21 5.89 mm to (49.3, 86.0)
- moved LED1 5.89 mm to (126.6, 141.8)
- moved LED7 5.89 mm to (127.1, 86.8)
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- renumbered C1 to C11, C2 to C12, C3 to C13, C4 to C14, C5 to C15, C6 to C16, C7 to C17, C8 to C18, C9 to C19, C10 to C20, C11 to C21, C12 to C22, C13 to C23, C14 to C24, C15 to C25, C16 to C26, C17 to C27, R6 to R10, R7 to R11, R8 to R12, R9 to R13, R10 to R14, R11 to R15, R12 to R16, R13 to R17, R14 to R18, R15 to R19, R16 to R20, R17 to R21, R18 to R22, R19 to R23, R20 to R24, R21 to R25, R22 to R26, R23 to R27, R24 to R28, R25 to R29, R3 to R5, R4 to R7, R5 to R9
Connections:
- U1 pad 1: unconnected-(U1-L1-Pad1) -> Net-(U1-L1)
- U1 pad 10: unconnected-(U1-L2-Pad10) -> Net-(U1-L2)
- U1 pad 11: unconnected-(U1-PGND-Pad11) -> GND
- U1 pad 3: unconnected-(U1-EN-Pad3) -> Net-(PWR1-Pin_1)
- U1 pad 4: unconnected-(U1-PS/SYNC-Pad4) -> GND
- U1 pad 5: unconnected-(U1-PG-Pad5) -> Net-(U1-PG)
- U1 pad 6: unconnected-(U1-VAUX-Pad6) -> Net-(U1-VAUX)
- U1 pad 8: unconnected-(U1-FB-Pad8) -> Net-(U1-FB)
- U2 pad 3: unconnected-(U2-EN-Pad3) -> Net-(U2-EN)
- U4 pad 3: +5V -> Net-(U4-Vs)
Routing:
- net Net-(U1-FB): track 0.00 -> 9.42 mm
- net Net-(PWR1-Pin_1): track 0.00 -> 7.55 mm
- net Net-(U1-L2): track 0.00 -> 4.22 mm
- net Net-(U1-L1): track 0.00 -> 4.20 mm
- net Net-(U1-VAUX): track 0.00 -> 2.69 mm
- net Net-(U1-PG): track 0.00 -> 2.58 mm
Other:
- outline, holes or cut-outs redrawn

Commit message: Up
Parts:
- moved PWR1 16.6 mm to (108.6, 43.5)
- moved C7 11.7 mm to (124.1, 40.7)
- moved C8 11.7 mm to (121.1, 40.7)
- moved C9 11.7 mm to (118.1, 40.7)
- moved R30 8.25 mm to (116.5, 52.4)
- moved U2 8.00 mm to (115.5, 48.8)
- moved C3 7.82 mm to (112.3, 46.8)
- moved C5 7.82 mm to (116.5, 45.0)
- moved C2 6.40 mm to (134.0, 44.6)
- moved L1 6.40 mm to (129.1, 40.5)
- moved R4 6.40 mm to (124.4, 50.1)
- moved C4 6.40 mm to (126.7, 50.1)
- moved C6 6.40 mm to (122.2, 50.1)
- moved R3 6.40 mm to (123.0, 45.7)
- moved R6 6.40 mm to (130.8, 50.1)
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Routing:
- net port7: track 0.00 -> 192.8 mm, vias 0 -> 1
- net port8: track 0.00 -> 189.6 mm, vias 0 -> 1
- net dim4: track 0.00 -> 155.0 mm, vias 0 -> 2
- net Net-(U3-IO12): track 0.00 -> 132.2 mm
- net Net-(U3-IO25): track 0.00 -> 121.9 mm, vias 0 -> 1
- net Net-(U3-IO26): track 0.00 -> 116.6 mm, vias 0 -> 1
- net +5V: track 0.00 -> 114.1 mm, vias 0 -> 25
- net sensOut4: track 0.00 -> 111.7 mm
- net dim2: track 0.00 -> 110.4 mm
- net dim1: track 0.00 -> 110.2 mm
- net port1: track 0.00 -> 109.4 mm
- net dim3: track 0.00 -> 107.6 mm
- net port2: track 0.00 -> 103.6 mm
- net sensOut3: track 0.00 -> 102.2 mm
- net port3: track 0.00 -> 95.2 mm
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- added copper zone on In2.Cu, net +3.3V
- added copper zone on In1.Cu, net +5V
- added copper zone on B.Cu, net GND
- added copper zone on F.Cu, net GND

Commit message: up
Parts:
- U1: footprint Package_SON:Texas_S-PWSON-N10_ThermalVias -> Package_SON:Texas_DSC0010J_ThermalVias
